File: hardware/eps/kicad/Solar_Charger.kicad_sch (KiCad schematic)
At the start: 32 parts, among them J1 B2B-PH-K-S(LF)(SN), J2 B2B-PH-K-S(LF)(SN), J3 B2B-PH-K-S(LF)(SN), J4 B2B-PH-K-S(LF)(SN), J5 B2B-PH-K-S(LF)(SN), J6 B2B-PH-K-S(LF)(SN), J7 TSW-103-07-F-S, J8 68000-102HLF, Q1 FDMC8327L, Q2 FDMC8327L, U1 LTC4162EUFD-LADMTRPBF

Commit message: attempt to convert altium to kicad, lost foot prints, not good
Parts:
- U6: renamed from U1; DATASHEET https://www.analog.com/media/en/technical-documentation/dat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 -> (none)
- renumbered C9 to C45, C3 to C46, C1 to C47, C2 to C48, C4 to C49, C5 to C50, C6 to C51, C7 to C52, D1 to D2, J1 to J11, J2 to J12, J3 to J13, J4 to J14, J5 to J15, J6 to J16, J7 to J17, J8 to J18, L1 to L6, Q1 to Q3, Q2 to Q4, R9 to R28, R1 to R29, R2 to R30, R4 to R31, R3 to R32, R5 to R33, R6 to R34, R8 to R35, R7 to R36, RS1 to RS3, RS2 to RS4
Other:
- note removed: "${##}"
- note removed: "${#}"
- note removed: "${DRAWNBY}"
- note removed: "${REVISION}"
- note removed: "${TITLE}"
- moved on the sheet: C45, C46, C47, C48, C49, C50, C51, C52, D2, J11, J12, J13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

Commit message: eps/kicad: assemble the schematic hierarchy and link it to the PCB
  The three .kicad_sch files were independent roots from the Altium import.
  Opening the project showed only the root's 17 components; the other 60
  were in files KiCad had no path to. Separately, the PCB shared no UUIDs
  at all with any schematic -- it had been imported independently, so the
  board-to-schematic link did not exist rather than being broken.

  Both are now fixed. Root sheet carries sheet symbols for Regulation and
  Solar_Charger, and all 77 footprints link to their symbols: 17 on the
  root, 28 in Regulation, 32 in Solar_Charger, matching the schematics
  exactly. Sheet-local nets picked up hierarchical paths, which cleared
  the "via connected to unknown net" warnings.

  Getting there took several passes and two things had to be repaired
  first.

  Annotation. Building the hierarchy in KiCad re-annotated the child
  sheets -- Solar_Charger went J1-J8 to J11-J18, C1-C24 became C41-C52 --
  because a duplicate J5 blocked the assembly. The refdes are the only
  link to the board, so 69 footprints were deleted as orphans. Every
  symbol UUID survived, so the old annotation was restored exactly by
  UUID, and the board was restored from the previous commit. The J5
  collision is resolved properly: J5 is the JST connector, and the XT30
  that shared its designator is now J10, on both the schematic and the
  board.

  Footprint fields. The import left them unusable -- only 5 of 40 carried
  a library prefix, and 10 pointed at
  C__Users_dng_Documents_AltiumLL_SamacSys.PcbLib, a Windows path from the
  machine that ran the import. All 77 are now the board's own qualified
  ids, which removed about 60 "missing a library name" warnings per
  update.

  The last 11 footprints would not link no matter how the update dialog
  was configured: KiCad matched 66 by UUID path and never fell back to
  reference designators for the remainder. Their paths were written
  directly instead, following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
Parts:
- C1: renamed from C47; footprint FP-GRM188-0_1-e0_2_0_55-IPC_A -> Vault:FP-GRM188-0_1-e0_2_0_55-IPC_A
- C2: renamed from C48; footprint CAPC1005X56X25ML10T15 -> Vault:CAPC1005X56X25ML10T15
- C3: renamed from C46; footprint C__Users_dng_Documents_AltiumLL_SamacSys.PcbLib:CAPC1005X56N -> SamacSys:CAPC1005X56N
- C4: renamed from C49; footprint C__Users_dng_Documents_AltiumLL_SamacSys.PcbLib:CAPC1005X56N -> SamacSys:CAPC1005X56N
- C5: renamed from C50; footprint FP-1206-L_3_2_0_3-W_1_6_0-IPC_A -> Vault:FP-1206-L_3_2_0_3-W_1_6_0-IPC_A
- C6: renamed from C51; footprint FP-CC0402-MFG -> Vault:FP-CC0402-MFG
- C7: renamed from C52; footprint FP-1206-L_3_2_0_3-W_1_6_0-IPC_A -> Vault:FP-1206-L_3_2_0_3-W_1_6_0-IPC_A
- C9: renamed from C45; footprint C__Users_dng_Documents_AltiumLL_SamacSys.PcbLib:EEE0JA152UAP -> SamacSys:EEE0JA152UAP
- D1: renamed from D2; footprint WL-SMCW_0603_150060xx75000 -> Vault:WL-SMCW_0603_150060xx75000
- J1: renamed from J11; footprint JST-B2B-PH-K-S_V -> Vault:JST-B2B-PH-K-S_V
- J2: renamed from J12; footprint JST-B2B-PH-K-S_V -> Vault:JST-B2B-PH-K-S_V
- J3: renamed from J13; footprint JST-B2B-PH-K-S_V -> Vault:JST-B2B-PH-K-S_V
- J4: renamed from J14; footprint JST-B2B-PH-K-S_V -> Vault:JST-B2B-PH-K-S_V
- J5: renamed from J15; footprint JST-B2B-PH-K-S_V -> Vault:JST-B2B-PH-K-S_V
- J6: renamed from J16; footprint JST-B2B-PH-K-S_V -> Vault:JST-B2B-PH-K-S_V
- J7: renamed from J17; footprint SMTC-TSW-103-07-X-S -> Vault:SMTC-TSW-103-07-X-S
- J8: renamed from J18; footprint AMPH-68000-102HLF_V -> Vault:AMPH-68000-102HLF_V
- L1: renamed from L6; footprint C__Users_dng_Documents_AltiumLL_SamacSys.PcbLib:XAL6060682MEC -> SamacSys:XAL6060682MEC
- Q1: renamed from Q3; footprint WDFN8_511DR_OSI -> Vault:WDFN8_511DR_OSI
- Q2: renamed from Q4; footprint WDFN8_511DR_OSI -> Vault:WDFN8_511DR_OSI
- R1: renamed from R29; footprint FP-CRCW0402-e3-IPC_C -> Vault:FP-CRCW0402-e3-IPC_C
- R2: renamed from R30; footprint RESC1005X40X25NL05T05 -> Vault:RESC1005X40X25NL05T05
- R3: renamed from R32; footprint C__Users_dng_Documents_AltiumLL_SamacSys.PcbLib:RESC3116X65N -> SamacSys:RESC3116X65N
- R4: renamed from R31; footprint C__Users_dng_Documents_AltiumLL_SamacSys.PcbLib:RESC3116X65N -> SamacSys:RESC3116X65N
- R5: renamed from R33; footprint FP-CRCW0603-e3-MFG -> Vault:FP-CRCW0603-e3-MFG
- R6: renamed from R34; footprint FP-CRCW0603-e3-IPC_B -> Vault:FP-CRCW0603-e3-IPC_B
- R7: renamed from R36; footprint RESC1609X50X30NL8T20 -> Vault:RESC1609X50X30NL8T20
- R8: renamed from R35; footprint RESC1609X50X30NL8T20 -> Vault:RESC1609X50X30NL8T20
- R9: renamed from R28; footprint FP-RT0603-MFG -> Vault:FP-RT0603-MFG
- RS1: renamed from RS3; footprint FP-PRL0816-MFG -> Vault:FP-PRL0816-MFG
- RS2: renamed from RS4; footprint FP-PRL0816-MFG -> Vault:FP-PRL0816-MFG
- U1: renamed from U6; footprint 05-08-1712_ADI -> Vault:05-08-1712_ADI
