File: hardware/comms/kicad/Power.kicad_sch (KiCad schematic)
At the start: 10 parts

Commit message: Repair UHF/UHF comms schematic and document PCB blockers
Correct PSA4 LNA and Hottech transistor pin mappings, RX capacitor values, and BPSK net labeling.

Assign verified XOR, resistor, and test-point footprints. Correct bulk capacitor polarity and add Panasonic land patterns.

Add project RF libraries, pin-map audit, and TOOD checklist. Record unresolved library loading, connectivity export, and PCB synchronization issues.
Parts:
- C58, C59: footprint (none) -> Ember_RF:CP_Elec_Panasonic_D_6.3x5.8; symbol Device:C_US -> Device:C_Polarized_US; MPN (none) -> EEHZA1V470P; Manufacturer (none) -> Panasonic; Voltage (none) -> 35V
Changed lines of the file:
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@@
 		(title "CubeSat Comms -- Power")
 		(rev "A")
+		(comment 9 "UHF/UHF revision in review - not for fabrication")
 	)
 	(rectangle
@@
 	)
 	(symbol
-		(lib_id "Device:C_US")
+		(lib_id "Device:C_Polarized_US")
 		(at 76.2 97.79 0)
 		(unit 1)
@@
 			)
 		)
-		(property "Footprint" ""
+		(property "Footprint" "Ember_RF:CP_Elec_Panasonic_D_6.3x5.8"
 			(at 76.2 97.79 0)
 			(hide yes)
@@
 			)
 		)
-		(property "Datasheet" ""
+		(property "Datasheet" "https://industrial.panasonic.com/content/data/CP/PDF/news2014/en/VH_E.pdf"
 			(at 76.2 97.79 0)
 			(hide yes)
@@
 			)
 		)
-		(property "Description" "capacitor, US symbol"
+		(property "Description" "47uF 35V polarized hybrid aluminum electrolytic; ZA size D"
 			(at 76.2 97.79 0)
 			(hide yes)
@@
 			)
 		)
-	)
+		(property "MPN" "EEHZA1V470P"
+			(at 76.2 97.79 0)
+			(hide yes)
+			(effects
+				(font
+					(size 1.27 1.27)
+				)
+			)
+		)
+		(property "Manufacturer" "Panasonic"
+			(at 76.2 97.79 0)
+			(hide yes)
+			(effects
+				(font
+					(size 1.27 1.27)
+				)
+			)
+		)
+		(property "Voltage" "35V"
+			(at 76.2 97.79 0)
+			(hide yes)
+			(effects
+				(font
+					(size 1.27 1.27)
+				)
+			)
+		))
 	(symbol
-		(lib_id "Device:C_US")
+		(lib_id "Device:C_Polarized_US")
 		(at 76.2 127 0)
 		(unit 1)
@@
 			)
 		)
-		(property "Footprint" ""
+		(property "Footprint" "Ember_RF:CP_Elec_Panasonic_D_6.3x5.8"
 			(at 76.2 127 0)
 			(hide yes)
@@
 			)
 		)
-		(property "Datasheet" ""
+		(property "Datasheet" "https://industrial.panasonic.com/content/data/CP/PDF/news2014/en/VH_E.pdf"
 			(at 76.2 127 0)
 			(hide yes)
@@
 			)
 		)
-		(property "Description" "capacitor, US symbol"
+		(property "Description" "47uF 35V polarized hybrid aluminum electrolytic; ZA size D"
 			(at 76.2 127 0)
 			(hide yes)
@@
 			)
 		)
-	)
+		(property "MPN" "EEHZA1V470P"
+			(at 76.2 127 0)
+			(hide yes)
+			(effects
+				(font
+					(size 1.27 1.27)
+				)
+			)
+		)
+		(property "Manufacturer" "Panasonic"
+			(at 76.2 127 0)
+			(hide yes)
+			(effects
+				(font
+					(size 1.27 1.27)
+				)
+			)
+		)
+		(property "Voltage" "35V"
+			(at 76.2 127 0)
+			(hide yes)
+			(effects
+				(font
+					(size 1.27 1.27)
+				)
+			)
+		))
 	(symbol
 		(lib_id "power:+3V3")
