File: hardware/comms/kicad/transceiver.kicad_sch (KiCad schematic)
At the start: 0 parts

Commit message: Repair UHF/UHF comms schematic and document PCB blockers
Correct PSA4 LNA and Hottech transistor pin mappings, RX capacitor values, and BPSK net labeling.

Assign verified XOR, resistor, and test-point footprints. Correct bulk capacitor polarity and add Panasonic land patterns.

Add project RF libraries, pin-map audit, and TOOD checklist. Record unresolved library loading, connectivity export, and PCB synchronization issues.
Other:
- title: CubeSat Comms -- Overview -> CubeSat Comms -- UHF/UHF Overview
Changed lines of the file:
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@@
 	(paper "A3")
 	(title_block
-		(title "CubeSat Comms -- Overview")
+		(title "CubeSat Comms -- UHF/UHF Overview")
 		(rev "A")
+		(comment 9 "UHF/UHF revision in review - not for fabrication")
 	)
 	(rectangle

Commit message: Checkpoint validated single-antenna comms routing before placement optimization
Other:
- added sheet Single Antenna RF Switch (RF_Switch.kicad_sch)
Changed lines of the file:
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@@
+	)
+	(sheet
+		(at 326.39 25.4)
+		(size 54.61 22.86)
+		(exclude_from_sim no)
+		(in_bom yes)
+		(on_board yes)
+		(dnp no)
+		(fields_autoplaced yes)
+		(stroke
+			(width 0.1524)
+			(type solid)
+		)
+		(fill
+			(color 0 0 0 0)
+		)
+		(property "Sheetname" "Single Antenna RF Switch"
+			(at 326.39 24.765 0)
+			(show_name no)
+			(do_not_autoplace no)
+			(effects
+				(font
+					(size 1.27 1.27)
+				)
+				(justify left bottom)
+			)
+		)
+		(property "Sheetfile" "RF_Switch.kicad_sch"
+			(at 326.39 48.895 0)
+			(show_name no)
+			(do_not_autoplace no)
+			(effects
+				(font
+					(size 1.27 1.27)
+				)
+				(justify left top)
+			)
+		)
 	)
 	(sheet
