File: hardware/comms/kicad/Clock_Gen.kicad_sch (KiCad schematic)
At the start: 13 parts, among them Y1 25MHz, Y2 Si5351A-B-GT

Commit message: progress on comms board
Parts:
- Y2: LCSC Part # (none) -> C504891; Manufacturer Part # (none) -> SI5351A-B-GTR
Changed lines of the file:
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@@
+			)
+		)
+		(property "LCSC Part #" "C504891"
+			(at 135.89 118.11 0)
+			(hide yes)
+			(show_name no)
+			(do_not_autoplace no)
+			(effects
+				(font
+					(size 1.27 1.27)
+				)
+			)
+		)
+		(property "Manufacturer Part #" "SI5351A-B-GTR"
+			(at 135.89 118.11 0)
+			(hide yes)
+			(show_name no)
+			(do_not_autoplace no)
+			(effects
+				(font
+					(size 1.27 1.27)
+				)
 			)
 		)
