File: hardware/comms/kicad/Clock_Gen.kicad_sch (KiCad schematic)
At the start: 13 parts, among them Y1 Crystal_GND2, Y2 Si5351A-B-GT

Commit message: comms: checkpoint current KiCad design before ground station work
Parts:
- R3, R4: footprint (none) -> Resistor_SMD:R_0402_1005Metric; Manufacturer (none) -> YAGEO; Manufacturer Part # (none) -> RC0402JR-070RL
- Y1: value Crystal_GND2 -> 25MHz; symbol Device:Crystal_GND2 -> Device:Crystal_GND24; MPN (none) -> ABM8G-25.000MHZ-B4Y-T; Manufacturer (none) -> Abracon
- Y2: LCSC Part # (none) -> C504891; Manufacturer Part # (none) -> SI5351A-B-GTR
Connections:
- net GND: now also Y1.4 (G)
Changed lines of the file:
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@@
 		(title "CubeSat Comms -- Clock Generator")
 		(rev "A")
+		(comment 9 "UHF/UHF revision in review - not for fabrication")
 	)
 	(rectangle
@@
 			)
 		)
-		(property "Footprint" ""
+		(property "Footprint" "Resistor_SMD:R_0402_1005Metric"
 			(at 187.96 112.268 90)
 			(hide yes)
@@
 			)
 		)
-		(property "Manufacturer Part #" ""
+		(property "Manufacturer Part #" "RC0402JR-070RL"
 			(at 187.96 110.49 90)
 			(hide yes)
@@
 		(property "LCSC Part #" "C60485"
 			(at 194.31 115.316 90)
+			(show_name no)
+			(do_not_autoplace no)
+			(effects
+				(font
+					(size 1.27 1.27)
+				)
+			)
+		)
+		(property "Manufacturer" "YAGEO"
+			(at 187.96 110.49 0)
+			(hide yes)
 			(show_name no)
 			(do_not_autoplace no)
@@
 			)
 		)
-		(property "Footprint" ""
+		(property "Footprint" "Resistor_SMD:R_0402_1005Metric"
 			(at 187.96 121.158 90)
 			(hide yes)
@@
 			)
 		)
-		(property "Manufacturer Part #" ""
+		(property "Manufacturer Part #" "RC0402JR-070RL"
 			(at 187.96 119.38 90)
 			(hide yes)
@@
 		(property "LCSC Part #" "C60485"
 			(at 194.31 124.206 90)
+			(show_name no)
+			(do_not_autoplace no)
+			(effects
+				(font
+					(size 1.27 1.27)
+				)
+			)
+		)
+		(property "Manufacturer" "YAGEO"
+			(at 187.96 119.38 0)
+			(hide yes)
 			(show_name no)
 			(do_not_autoplace no)
@@
 			)
 		)
+		(property "LCSC Part #" "C504891"
+			(at 135.89 118.11 0)
+			(hide yes)
+			(show_name no)
+			(do_not_autoplace no)
+			(effects
+				(font
+					(size 1.27 1.27)
+				)
+			)
+		)
+		(property "Manufacturer Part #" "SI5351A-B-GTR"
+			(at 135.89 118.11 0)
+			(hide yes)
+			(show_name no)
+			(do_not_autoplace no)
+			(effects
+				(font
+					(size 1.27 1.27)
+				)
+			)
+		)
 		(pin "3"
 		)
@@
 	)
 	(symbol
-		(lib_id "Device:Crystal_GND2")
+		(lib_id "Device:Crystal_GND24")
 		(at 87.63 111.76 270)
 		(unit 1)
@@
 			)
 		)
-		(property "Value" "Crystal_GND2"
+		(property "Value" "25MHz"
 			(at 91.44 113.0299 90)
 			(show_name no)
@@
 			)
 		)
-		(property "Datasheet" ""
+		(property "Datasheet" "https://abracon.com/Resonators/ABM8G.pdf"
 			(at 87.63 111.76 0)
 			(hide yes)
@@
 			)
 		)
-		(property "Description" "Three pin crystal, GND on pin 2"
+		(property "Description" "25 MHz four-pad crystal; pins 2 and 4 ground"
 			(at 87.63 111.76 0)
 			(hide yes)
@@
 			)
 		)
+		(property "MPN" "ABM8G-25.000MHZ-B4Y-T"
+			(at 87.63 111.76 0)
+			(hide yes)
+			(show_name no)
+			(do_not_autoplace no)
+			(effects
+				(font
+					(size 1.27 1.27)
+				)
+			)
+		)
+		(property "Manufacturer" "Abracon"
+			(at 87.63 111.76 0)
+			(hide yes)
+			(show_name no)
+			(do_not_autoplace no)
+			(effects
+				(font
+					(size 1.27 1.27)
+				)
+			)
+		)
 		(pin "2"
 		)
@@
 		(pin "1"
 		)
+		(pin "4"
+		)
 		(instances
