File: hardware/comms/kicad/Connectors.kicad_sch (KiCad schematic)
At the start: 13 parts, among them J9 Conn_Coaxial_Small

Commit message: Repair UHF/UHF comms schematic and document PCB blockers
Correct PSA4 LNA and Hottech transistor pin mappings, RX capacitor values, and BPSK net labeling.

Assign verified XOR, resistor, and test-point footprints. Correct bulk capacitor polarity and add Panasonic land patterns.

Add project RF libraries, pin-map audit, and TOOD checklist. Record unresolved library loading, connectivity export, and PCB synchronization issues.
Parts:
- TP11, TP12, TP13, TP14, TP15, TP16: footprint (none) -> TestPoint:TestPoint_Pad_D1.0mm
Changed lines of the file:
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@@
 		(title "CubeSat Comms - Connectors")
 		(rev "A")
+		(comment 9 "UHF/UHF revision in review - not for fabrication")
 	)
 	(rectangle
@@
 			)
 		)
-		(property "Footprint" ""
+		(property "Footprint" "TestPoint:TestPoint_Pad_D1.0mm"
 			(at 110.49 167.64 0)
 			(hide yes)
@@
 			)
 		)
-		(property "Footprint" ""
+		(property "Footprint" "TestPoint:TestPoint_Pad_D1.0mm"
 			(at 110.49 177.8 0)
 			(hide yes)
@@
 			)
 		)
-		(property "Footprint" ""
+		(property "Footprint" "TestPoint:TestPoint_Pad_D1.0mm"
 			(at 110.49 182.88 0)
 			(hide yes)
@@
 			)
 		)
-		(property "Footprint" ""
+		(property "Footprint" "TestPoint:TestPoint_Pad_D1.0mm"
 			(at 110.49 187.96 0)
 			(hide yes)
@@
 			)
 		)
-		(property "Footprint" ""
+		(property "Footprint" "TestPoint:TestPoint_Pad_D1.0mm"
 			(at 110.49 172.72 0)
 			(hide yes)
@@
 			)
 		)
-		(property "Footprint" ""
+		(property "Footprint" "TestPoint:TestPoint_Pad_D1.0mm"
 			(at 110.49 193.04 0)
 			(hide yes)

Commit message: Checkpoint comms PCB synchronization and connector alignment
Repair schematic-to-PCB links and apply the native update. Standardize J6/J7/J8 as DNP headers, align CSKB sockets for top-side assembly, and record pad-mapping verification.

Pre-RF-layout checkpoint: retain legacy circuitry for reviewed cleanup. Latest DRC has 631 errors, 273 warnings, and 140 unconnected items; board is not fabrication-ready.
Parts:
- H3, H4: footprint (none) -> Ember_RF:Samtec_ESQ-126-39-G-D_2x26_P2.54mm; MPN (none) -> ESQ-126-39-G-D; Manufacturer (none) -> Samtec
Changed lines of the file:
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@@
 			)
 		)
-		(property "Footprint" ""
+		(property "Footprint" "Ember_RF:Samtec_ESQ-126-39-G-D_2x26_P2.54mm"
 			(at 259.08 106.68 0)
 			(hide yes)
@@
 			)
 		)
-		(property "Datasheet" ""
+		(property "Datasheet" "https://suddendocs.samtec.com/prints/esq-1xx-xx-x-x-xxx-xx-x-xx-mkt.pdf"
 			(at 259.08 106.68 0)
 			(hide yes)
@@
 		)
 		(property "Description" "Generic connector, double row, 02x26, odd/even pin numbering scheme (row 1 odd numbers, row 2 even numbers), script generated (kicad-library-utils/schlib/autogen/connector/)"
+			(at 259.08 106.68 0)
+			(hide yes)
+			(show_name no)
+			(do_not_autoplace no)
+			(effects
+				(font
+					(size 1.27 1.27)
+				)
+			)
+		)
+		(property "MPN" "ESQ-126-39-G-D"
+			(at 259.08 106.68 0)
+			(hide yes)
+			(show_name no)
+			(do_not_autoplace no)
+			(effects
+				(font
+					(size 1.27 1.27)
+				)
+			)
+		)
+		(property "Manufacturer" "Samtec"
 			(at 259.08 106.68 0)
 			(hide yes)
@@
 			)
 		)
-		(property "Footprint" ""
+		(property "Footprint" "Ember_RF:Samtec_ESQ-126-39-G-D_2x26_P2.54mm"
 			(at 132.08 106.68 0)
 			(hide yes)
@@
 			)
 		)
-		(property "Datasheet" ""
+		(property "Datasheet" "https://suddendocs.samtec.com/prints/esq-1xx-xx-x-x-xxx-xx-x-xx-mkt.pdf"
 			(at 132.08 106.68 0)
 			(hide yes)
@@
 			(at 132.08 106.68 0)
 			(hide yes)
+			(show_name no)
+			(do_not_autoplace no)
+			(effects
+				(font
+					(size 1.27 1.27)
+				)
+			)
+		)
+		(property "MPN" "ESQ-126-39-G-D"
+			(at 132.08 106.68 0)
+			(hide yes)
+			(show_name no)
+			(do_not_autoplace no)
+			(effects
+				(font
+					(size 1.27 1.27)
+				)
+			)
+		)
+		(property "Manufacturer" "Samtec"
+			(at 132.08 106.68 0)
+			(hide yes)

Commit message: progress on comms board
Parts:
- H1: renamed from H3; LCSC Part # (none) -> C7466599; Manufacturer Part # (none) -> ESQ-126-39-G-D
- H2: renamed from H4; LCSC Part # (none) -> C7466599; Manufacturer Part # (none) -> ESQ-126-39-G-D
- renumbered TP11 to TP1, TP12 to TP2, TP13 to TP3, TP14 to TP4, TP15 to TP5, TP16 to TP6
Connections:
- net CAN_A_L: now reaches H1.1 (Pin_1)
- net CAN_B_L: now reaches H1.2 (Pin_2)
- net CAN_A_H: now reaches H1.3 (Pin_3)
- net CAN_B_H: now reaches H1.4 (Pin_4)
- net COMMS_IRQ: no longer names the net of H1.16 (Pin_16)
- net SPI_COMMS_CS_N: no longer names the net of H1.24 (Pin_24)
- net SPI_COMMS_MISO: no longer names the net of H1.22 (Pin_22)
- net SPI_COMMS_MOSI: no longer names the net of H1.23 (Pin_23)
- net SPI_COMMS_SCK: no longer names the net of H1.21 (Pin_21)
