File: hardware/comms/kicad/RX_Chain.kicad_sch (KiCad schematic)
At the start: 40 parts, among them Q4 2SC3356, U10 ADE-1+, U5 MCP6022, U9 PSA4-5043+

Commit message: Repair UHF/UHF comms schematic and document PCB blockers
Correct PSA4 LNA and Hottech transistor pin mappings, RX capacitor values, and BPSK net labeling.

Assign verified XOR, resistor, and test-point footprints. Correct bulk capacitor polarity and add Panasonic land patterns.

Add project RF libraries, pin-map audit, and TOOD checklist. Record unresolved library loading, connectivity export, and PCB synchronization issues.
Parts:
- C75: value C -> 100n; footprint (none) -> Capacitor_SMD:C_0402_1005Metric; LCSC Part # (none) -> C1525; Manufacturer Part # (none) -> CL05B104KO5NNNC
- C82: value 8.2p -> 100n; LCSC Part # C1579 -> C1525; Manufacturer Part # (none) -> CL05B104KO5NNNC
- C85: value 100n -> 8.2p; LCSC Part # C1525 -> C1579; Manufacturer Part # CL05B104KO5NNNC -> (none)
- Q4: symbol Simulation_SPICE:NPN -> Transistor_BJT:Q_NPN_BEC; Manufacturer (none) -> Guangdong Hottech; Manufacturer Part # (none) -> 2SC3356
- U9: footprint Package_TO_SOT_SMD:SOT-343_SC-70-4 -> Ember_RF:PSA4-5043_MMM1362; symbol RF_Amplifier:SPF5189Z -> Ember_RF:PSA4-5043+; MPN (none) -> PSA4-5043+; Manufacturer (none) -> Mini-Circuits
Connections:
- net GND: now also Q4.2 (E), U9.4 (GND); no longer Q4.3 (E)
- net at C85.1, C86.1, L18.2: now also Q4.3 (C); no longer Q4.1 (C)
- net at C83.1, R33.1: now also Q4.1 (B); no longer Q4.2 (B)
- net at C75.1, L16.2: now also U9.1 (OUT_DC); no longer U9.3
- net at C67.2: now also U9.3 (IN); no longer U9.1
Changed lines of the file:
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@@
 		(title "CubeSat Comms -- RX Chain")
 		(rev "A")
+		(comment 9 "UHF/UHF revision in review - not for fabrication")
 	)
 	(rectangle
@@
 	(wire
 		(pts
+			(xy 152.4 86.36) (xy 147.32 86.36)
+		)
+		(stroke
+			(width 0)
+			(type default)
+		)
+	)
+	(wire
+		(pts
 			(xy 195.58 105.41) (xy 199.39 105.41)
 		)
@@
 	(wire
 		(pts
+			(xy 161.29 73.66) (xy 165.1 73.66)
+		)
+		(stroke
+			(width 0)
+			(type default)
+		)
+	)
+	(wire
+		(pts
 			(xy 289.56 85.09) (xy 294.64 85.09)
 		)
@@
 	(wire
 		(pts
-			(xy 157.48 73.66) (xy 165.1 73.66)
+			(xy 133.35 73.66) (xy 138.43 73.66)
 		)
 		(stroke
@@
 	(wire
 		(pts
+			(xy 152.4 81.28) (xy 152.4 86.36)
+		)
+		(stroke
+			(width 0)
+			(type default)
+		)
+	)
+	(wire
+		(pts
 			(xy 124.46 184.15) (xy 132.08 184.15)
 		)
@@
 	(wire
 		(pts
-			(xy 133.35 73.66) (xy 142.24 73.66)
-		)
-		(stroke
-			(width 0)
-			(type default)
-		)
-	)
-	(wire
-		(pts
 			(xy 248.92 99.06) (xy 248.92 101.6)
 		)
@@
 		(shape output)
 		(at 335.28 110.49 0)
-		(fields_autoplaced yes)
 		(effects
 			(font
@@
 		(shape bidirectional)
 		(at 195.58 105.41 180)
-		(fields_autoplaced yes)
 		(effects
 			(font
@@
 		(shape input)
 		(at 39.37 100.33 180)
-		(fields_autoplaced yes)
 		(effects
 			(font
@@
 		(shape input)
 		(at 50.8 186.69 180)
-		(fields_autoplaced yes)
 		(effects
 			(font
@@
 		(shape output)
 		(at 256.54 193.04 0)
-		(fields_autoplaced yes)
 		(effects
 			(font
@@
 			)
 		)
-		(property "Value" "8.2p"
+		(property "Value" "100n"
 			(at 204.216 90.424 0)
 			(show_name no)
@@
 			)
 		)
-		(property "LCSC Part #" "C1579"
+		(property "LCSC Part #" "C1525"
 			(at 202.946 92.202 0)
 			(show_name no)
@@
 			)
 		)
+		(property "Manufacturer Part #" "CL05B104KO5NNNC"
+			(at 199.39 86.36 0)
+			(hide yes)
+			(show_name no)
+			(do_not_autoplace no)
+			(effects
+				(font
+					(size 1.27 1.27)
+				)
+			)
+		)
 		(pin "2"
 		)
@@
 	)
 	(symbol
-		(lib_id "RF_Amplifier:SPF5189Z")
+		(lib_id "Ember_RF:PSA4-5043+")
 		(at 149.86 73.66 0)
 		(unit 1)
@@
 		(dnp no)
 		(property "Reference" "U9"
-			(at 152.146 77.216 0)
+			(at 149.86 68.58 0)
 			(show_name no)
 			(do_not_autoplace no)
@@
 		)
 		(property "Value" "PSA4-5043+"
-			(at 157.226 79.248 0)
+			(at 149.86 81.28 0)
 			(show_name no)
 			(do_not_autoplace no)
@@
 			)
 		)
-		(property "Footprint" "Package_TO_SOT_SMD:SOT-343_SC-70-4"
+		(property "Footprint" "Ember_RF:PSA4-5043_MMM1362"
 			(at 151.13 63.5 0)
 			(hide yes)
@@
 			)
 		)
-		(property "Datasheet" "www.qorvo.com/products/d/da001910"
+		(property "Datasheet" "https://www.minicircuits.com/pdfs/PSA4-5043+.pdf"
 			(at 149.86 73.66 0)
 			(hide yes)
@@
 			)
 		)
-		(property "Description" "50MHz to 4000MHz, GaAs pHEMT low noise MMIC amplifier, SOT-89"
+		(property "Description" "Mini-Circuits PSA4-5043+ low-noise RF amplifier, MMM1362 SOT-343; pin 3 IN, pin 1 OUT/DC, pins 2/4 GND"
 			(at 149.86 73.66 0)
 			(hide yes)
@@
 			)
 		)
+		(property "MPN" "PSA4-5043+"
+			(at 149.86 73.66 0)
+			(hide yes)
+			(show_name no)
+			(do_not_autoplace no)
+			(effects
+				(font
+					(size 1.27 1.27)
+				)
+			)
+		)
+		(property "Manufacturer" "Mini-Circuits"
+			(at 149.86 73.66 0)
+			(hide yes)
+			(show_name no)
+			(do_not_autoplace no)
+			(effects
+				(font
+					(size 1.27 1.27)
+				)
+			)
+		)
 		(pin "2"
 		)
@@
 		(pin "1"
 		)
+		(pin "4"
+		)
 		(instances
 			(project "transceiver"
@@
 			)
 		)
-		(property "Value" "C"
+		(property "Value" "100n"
 			(at 176.022 76.708 90)
 			(show_name no)
@@
 			)
 		)
-		(property "Footprint" ""
+		(property "Footprint" "Capacitor_SMD:C_0402_1005Metric"
 			(at 177.8 72.6948 0)
 			(hide yes)
@@
 			)
 		)
+		(property "LCSC Part #" "C1525"
+			(at 173.99 73.66 0)
+			(hide yes)
+			(show_name no)
+			(do_not_autoplace no)
+			(effects
+				(font
+					(size 1.27 1.27)
+				)
+			)
+		)
+		(property "Manufacturer Part #" "CL05B104KO5NNNC"
+			(at 173.99 73.66 0)
+			(hide yes)
+			(show_name no)
+			(do_not_autoplace no)
+			(effects
+				(font
+					(size 1.27 1.27)
+				)
+			)
+		)
 		(pin "1"
 		)
@@
 			)
 		)
-		(property "Value" "100n"
+		(property "Value" "8.2p"
 			(at 221.742 90.678 0)
 			(show_name no)
@@
 			)
 		)
-		(property "LCSC Part #" "C1525"
+		(property "LCSC Part #" "C1579"
 			(at 222.504 92.71 0)
 			(show_name no)
@@
 			)
 		)
-		(property "Manufacturer Part #" "CL05B104KO5NNNC"
+		(property "Manufacturer Part #" ""
 			(at 218.44 86.36 90)
 			(hide yes)
@@
 	)
 	(symbol
-		(lib_id "Simulation_SPICE:NPN")
+		(lib_id "Transistor_BJT:Q_NPN_BEC")
 		(at 223.52 105.41 0)
 		(unit 1)
@@
 			)
 		)
-		(property "Datasheet" "https://ngspice.sourceforge.io/docs/ngspice-html-manual/manual.xhtml#cha_BJTs"
+		(property "Datasheet" "https://www.lcsc.com/datasheet/C193010.pdf"
 			(at 287.02 105.41 0)
 			(hide yes)
@@
 			)
 		)
-		(property "Description" "Bipolar transistor symbol for simulation only, substrate tied to the emitter"
+		(property "Description" "Hottech 2SC3356 SOT-23; B=1 E=2 C=3; do not substitute Renesas pinout"
 			(at 223.52 105.41 0)
 			(hide yes)
@@
 			)
 		)
-		(property "Sim.Pins" "1=C 2=B 3=E"
+		(property "Sim.Pins" "1=B 2=E 3=C"
 			(at 223.52 105.41 0)
 			(hide yes)
@@
 			(show_name no)
 			(do_not_autoplace no)
+			(effects
+				(font
+					(size 1.27 1.27)
+				)
+			)
+		)
+		(property "Manufacturer" "Guangdong Hottech"
+			(at 223.52 105.41 0)
+			(hide yes)
+			(show_name no)
+			(do_not_autoplace no)
+			(effects
+				(font
+					(size 1.27 1.27)
+				)
+			)
+		)
+		(property "Manufacturer Part #" "2SC3356"
+			(at 223.52 105.41 0)
+			(hide yes)
+			(show_name no)
+			(do_not_autoplace no)

Commit message: Checkpoint comms PCB synchronization and connector alignment
Repair schematic-to-PCB links and apply the native update. Standardize J6/J7/J8 as DNP headers, align CSKB sockets for top-side assembly, and record pad-mapping verification.

Pre-RF-layout checkpoint: retain legacy circuitry for reviewed cleanup. Latest DRC has 631 errors, 273 warnings, and 140 unconnected items; board is not fabrication-ready.
Parts:
- U5: footprint (none) -> Package_SO:SOIC-8_3.9x4.9mm_P1.27mm; MPN (none) -> MCP6022-I/SN; Manufacturer (none) -> Microchip Technology
Changed lines of the file:
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@@
 			)
 		)
-		(property "Footprint" ""
+		(property "Footprint" "Package_SO:SOIC-8_3.9x4.9mm_P1.27mm"
 			(at 116.84 184.15 0)
 			(hide yes)
@@
 			)
 		)
-		(property "Datasheet" "http://ww1.microchip.com/downloads/en/devicedoc/20001685e.pdf"
+		(property "Datasheet" "https://ww1.microchip.com/downloads/en/DeviceDoc/20001685E.pdf"
 			(at 116.84 184.15 0)
 			(hide yes)
@@
 			)
 		)
+		(property "MPN" "MCP6022-I/SN"
+			(at 116.84 184.15 0)
+			(hide yes)
+			(show_name no)
+			(do_not_autoplace no)
+			(effects
+				(font
+					(size 1.27 1.27)
+				)
+			)
+		)
+		(property "Manufacturer" "Microchip Technology"
+			(at 116.84 184.15 0)
+			(hide yes)
+			(show_name no)
+			(do_not_autoplace no)
+			(effects
+				(font
+					(size 1.27 1.27)
+				)
+			)
+		)
 		(pin "6"
 		)
@@
 			)
 		)
-		(property "Footprint" ""
+		(property "Footprint" "Package_SO:SOIC-8_3.9x4.9mm_P1.27mm"
 			(at 236.22 210.82 0)
 			(hide yes)
@@
 			)
 		)
-		(property "Datasheet" "http://ww1.microchip.com/downloads/en/devicedoc/20001685e.pdf"
+		(property "Datasheet" "https://ww1.microchip.com/downloads/en/DeviceDoc/20001685E.pdf"
 			(at 236.22 210.82 0)
 			(hide yes)
@@
 			)
 		)
+		(property "MPN" "MCP6022-I/SN"
+			(at 236.22 210.82 0)
+			(hide yes)
+			(show_name no)
+			(do_not_autoplace no)
+			(effects
+				(font
+					(size 1.27 1.27)
+				)
+			)
+		)
+		(property "Manufacturer" "Microchip Technology"
+			(at 236.22 210.82 0)
+			(hide yes)
+			(show_name no)
+			(do_not_autoplace no)
+			(effects
+				(font
+					(size 1.27 1.27)
+				)
+			)
+		)
 		(pin "4"
 		)
@@
 			)
 		)
-		(property "Footprint" ""
+		(property "Footprint" "Package_SO:SOIC-8_3.9x4.9mm_P1.27mm"
 			(at 215.9 191.77 0)
 			(hide yes)
@@
 			)
 		)
-		(property "Datasheet" "http://ww1.microchip.com/downloads/en/devicedoc/20001685e.pdf"
+		(property "Datasheet" "https://ww1.microchip.com/downloads/en/DeviceDoc/20001685E.pdf"
 			(at 215.9 191.77 0)
 			(hide yes)
@@
 			(at 215.9 191.77 0)
 			(hide yes)
+			(show_name no)
+			(do_not_autoplace no)
+			(effects
+				(font
+					(size 1.27 1.27)
+				)
+			)
+		)
+		(property "MPN" "MCP6022-I/SN"
+			(at 215.9 191.77 0)
+			(hide yes)
+			(show_name no)
+			(do_not_autoplace no)
+			(effects
+				(font
+					(size 1.27 1.27)
+				)
+			)
+		)
+		(property "Manufacturer" "Microchip Technology"
+			(at 215.9 191.77 0)
+			(hide yes)

Commit message: Checkpoint validated single-antenna comms routing before placement optimization
Parts:
- added R38, R39: 100k, Resistor_SMD:R_0402_1005Metric, symbol Device:R
- L16: value 1u -> 220n; footprint Inductor_SMD:L_0805_2012Metric -> Ember_RF:L_Coilcraft_0805HP; LCSC Part # C18221300 -> (none); MPN (none) -> 0805HP-221XJRC; Manufacturer (none) -> Coilcraft; Manufacturer Part # (none) -> 0805HP-221XJRC; PinMapAudit (none) -> design/l16_footprint_acceptance.md; Qualification (none) -> Prototype; RF bench qualification pending
- U10: MPN (none) -> ADE-1+; Manufacturer (none) -> Mini-Circuits; Package (none) -> CD636; PackageHeightMax_mm (none) -> 4.11; PinMapAudit (none) -> design/u10_ade1_pinmap.md
Connections:
- net GND: no longer R30.2
- net RX_IF: now also R38.1
- net RX_AMP_IN: now reaches C69.1, U5.5 (+)
- net RX_AMP_IN: now also R39.2; no longer C72.2
- net VREF_RX: now reaches R28.2, R29.1
- net VREF_RX: now also C72.2, R30.2, R38.2, R39.1

Commit message: progress on comms board
Parts:
- C83: LCSC Part # XXX -> C53547; Manufacturer Part # XXX -> 0402CG102J500NT
- U10: LCSC Part # (none) -> C2942210; Manufacturer Part # (none) -> ADE-1+
- U5: LCSC Part # (none) -> C57639; Manufacturer Part # (none) -> MCP6022T-I/SN
Changed lines of the file:
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@@
 			)
 		)
+		(property "LCSC Part #" "C57639"
+			(at 116.84 184.15 0)
+			(hide yes)
+			(show_name no)
+			(do_not_autoplace no)
+			(effects
+				(font
+					(size 1.27 1.27)
+				)
+			)
+		)
+		(property "Manufacturer Part #" "MCP6022T-I/SN"
+			(at 116.84 184.15 0)
+			(hide yes)
+			(show_name no)
+			(do_not_autoplace no)
+			(effects
+				(font
+					(size 1.27 1.27)
+				)
+			)
+		)
 		(pin "6"
 		)
@@
 			)
 		)
+		(property "LCSC Part #" "C57639"
+			(at 236.22 210.82 0)
+			(hide yes)
+			(show_name no)
+			(do_not_autoplace no)
+			(effects
+				(font
+					(size 1.27 1.27)
+				)
+			)
+		)
+		(property "Manufacturer Part #" "MCP6022T-I/SN"
+			(at 236.22 210.82 0)
+			(hide yes)
+			(show_name no)
+			(do_not_autoplace no)
+			(effects
+				(font
+					(size 1.27 1.27)
+				)
+			)
+		)
 		(pin "4"
 		)
@@
 			)
 		)
-		(property "LCSC Part #" "XXX"
+		(property "LCSC Part #" "C53547"
 			(at 203.962 112.522 90)
 			(show_name no)
@@
 			)
 		)
-		(property "Manufacturer Part #" "XXX"
+		(property "Manufacturer Part #" "0402CG102J500NT"
 			(at 203.2 105.41 90)
 			(hide yes)
@@
 			)
 		)
+		(property "LCSC Part #" "C57639"
+			(at 215.9 191.77 0)
+			(hide yes)
+			(show_name no)
+			(do_not_autoplace no)
+			(effects
+				(font
+					(size 1.27 1.27)
+				)
+			)
+		)
+		(property "Manufacturer Part #" "MCP6022T-I/SN"
+			(at 215.9 191.77 0)
+			(hide yes)
+			(show_name no)
+			(do_not_autoplace no)
+			(effects
+				(font
+					(size 1.27 1.27)
+				)
+			)
+		)
 		(pin "7"
 		)
@@
 			(at 320.04 85.09 0)
 			(hide yes)
+			(show_name no)
+			(do_not_autoplace no)
+			(effects
+				(font
+					(size 1.27 1.27)
+				)
+			)
+		)
+		(property "LCSC Part #" "C2942210"
+			(at 320.04 85.09 0)
+			(hide yes)
+			(show_name no)
+			(do_not_autoplace no)
+			(effects
+				(font
+					(size 1.27 1.27)
+				)
+			)
+		)
+		(property "Manufacturer Part #" "ADE-1+"
+			(at 320.04 85.09 0)
+			(hide yes)
