File: hardware/comms/kicad/TX_Chain.kicad_sch (KiCad schematic)
At the start: 28 parts, among them Q3 2SC3356, U7 74LVC1G86, U8 ADL5602ARKZ-R7

Commit message: comms: checkpoint current KiCad design before ground station work
Parts:
- Q3: symbol Simulation_SPICE:NPN -> Transistor_BJT:Q_NPN_BEC; Manufacturer (none) -> Guangdong Hottech; Manufacturer Part # (none) -> 2SC3356
- U7: footprint (none) -> Package_TO_SOT_SMD:SOT-23-5; MPN (none) -> SN74LVC1G86DBVR; Manufacturer (none) -> Texas Instruments
- U8: MPN (none) -> ADL5602ARKZ-R7; Manufacturer (none) -> Analog Devices; PinMapAudit (none) -> design/u8_adl5602_pinmap.md
Connections:
- net BPSK_DATA: no longer C73.2, U7.4
- net GND: now also Q3.2 (E); no longer Q3.3 (E)
- net TRIPLER_OUT: now also Q3.3 (C); no longer Q3.1 (C)
- net at C73.1, R27.1: now also Q3.1 (B); no longer Q3.2 (B)
- new net RF_TX_BPSK_145: C73.2, U7.4
Changed lines of the file:
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@@
 		(rev "B")
 		(comment 1 "Nick Grabbs - KI5YNG")
+		(comment 9 "UHF/UHF revision in review - not for fabrication")
 	)
 	(rectangle
@@
 		)
 	)
-	(global_label "CLK0_OUT"
-		(shape output)
-		(at 87.63 121.92 180)
-		(fields_autoplaced yes)
+	(label "RF_TX_BPSK_145"
+		(at 146.05 129.54 180)
 		(effects
 			(font
 				(size 1.27 1.27)
 			)
-			(justify right)
-		)
-		(property "Intersheetrefs" "${INTERSHEET_REFS}"
-			(at 75.271 121.92 0)
-			(hide yes)
-			(show_name no)
-			(do_not_autoplace no)
-			(effects
-				(font
-					(size 1.27 1.27)
-				)
-				(justify right)
-			)
+			(justify right bottom)
 		)
 	)
-	(global_label "BPSK_DATA"
+	(global_label "CLK0_OUT"
 		(shape output)
-		(at 146.05 129.54 180)
-		(fields_autoplaced yes)
+		(at 87.63 121.92 180)
 		(effects
 			(font
@@
 		)
 		(property "Intersheetrefs" "${INTERSHEET_REFS}"
-			(at 132.6629 129.54 0)
+			(at 75.271 121.92 0)
 			(hide yes)
 			(show_name no)
@@
 		(shape output)
 		(at 288.29 186.69 0)
-		(fields_autoplaced yes)
 		(effects
 			(font
@@
 		(shape output)
 		(at 87.63 127 180)
-		(fields_autoplaced yes)
 		(effects
 			(font
@@
 		(shape bidirectional)
 		(at 232.41 110.49 0)
-		(fields_autoplaced yes)
 		(effects
 			(font
@@
 		(shape input)
 		(at 107.95 200.66 180)
-		(fields_autoplaced yes)
 		(effects
 			(font
@@
 		(shape output)
 		(at 347.98 114.3 0)
-		(fields_autoplaced yes)
 		(effects
 			(font
@@
 	)
 	(symbol
-		(lib_id "Simulation_SPICE:NPN")
+		(lib_id "Transistor_BJT:Q_NPN_BEC")
 		(at 187.96 124.46 0)
 		(unit 1)
@@
 			)
 		)
-		(property "Datasheet" "https://ngspice.sourceforge.io/docs/ngspice-html-manual/manual.xhtml#cha_BJTs"
+		(property "Datasheet" "https://www.lcsc.com/datasheet/C193010.pdf"
 			(at 251.46 124.46 0)
 			(hide yes)
@@
 			)
 		)
-		(property "Description" "Bipolar transistor symbol for simulation only, substrate tied to the emitter"
+		(property "Description" "Hottech 2SC3356 SOT-23; B=1 E=2 C=3; do not substitute Renesas pinout"
 			(at 187.96 124.46 0)
 			(hide yes)
@@
 			)
 		)
-		(property "Sim.Pins" "1=C 2=B 3=E"
+		(property "Sim.Pins" "1=B 2=E 3=C"
 			(at 187.96 124.46 0)
 			(hide yes)
@@
 			)
 		)
+		(property "Manufacturer" "Guangdong Hottech"
+			(at 187.96 124.46 0)
+			(hide yes)
+			(show_name no)
+			(do_not_autoplace no)
+			(effects
+				(font
+					(size 1.27 1.27)
+				)
+			)
+		)
+		(property "Manufacturer Part #" "2SC3356"
+			(at 187.96 124.46 0)
+			(hide yes)
+			(show_name no)
+			(do_not_autoplace no)
+			(effects
+				(font
+					(size 1.27 1.27)
+				)
+			)
+		)
 		(pin "2"
 		)
@@
 			)
 		)
-		(property "Datasheet" "https://www.analog.com/media/en/technical-documentation/data-sheets/ADL5610.pdf"
+		(property "Datasheet" "https://www.analog.com/media/en/technical-documentation/data-sheets/ADL5602.pdf"
 			(at 123.19 200.66 0)
 			(hide yes)
@@
 			)
 		)
-		(property "Description" "30-6000MHz RF/IF +18.4dB gain block, SOT-89"
+		(property "Description" "ADL5602 50 MHz to 4 GHz RF/IF gain block, 20 dB nominal, 5 V, SOT-89; audited pin-compatible ADL5610 symbol"
 			(at 123.19 200.66 0)
 			(hide yes)
@@
 			)
 		)
+		(property "MPN" "ADL5602ARKZ-R7"
+			(at 123.19 200.66 0)
+			(hide yes)
+			(show_name no)
+			(do_not_autoplace no)
+			(effects
+				(font
+					(size 1.27 1.27)
+				)
+			)
+		)
+		(property "Manufacturer" "Analog Devices"
+			(at 123.19 200.66 0)
+			(hide yes)
+			(show_name no)
+			(do_not_autoplace no)
+			(effects
+				(font
+					(size 1.27 1.27)
+				)
+			)
+		)
+		(property "PinMapAudit" "design/u8_adl5602_pinmap.md"
+			(at 123.19 200.66 0)
+			(hide yes)
+			(show_name no)
+			(do_not_autoplace no)
+			(effects
+				(font
+					(size 1.27 1.27)
+				)
+			)
+		)
 		(pin "1"
 		)
@@
 			)
 		)
-		(property "Footprint" ""
+		(property "Footprint" "Package_TO_SOT_SMD:SOT-23-5"
 			(at 123.19 124.46 0)
 			(hide yes)
@@
 			)
 		)
-		(property "Datasheet" "http://www.ti.com/lit/sg/scyt129e/scyt129e.pdf"
+		(property "Datasheet" "https://www.ti.com/lit/ds/symlink/sn74lvc1g86.pdf"
 			(at 123.19 124.46 0)
 			(hide yes)
@@
 			(show_name no)
 			(do_not_autoplace no)
+			(effects
+				(font
+					(size 1.27 1.27)
+				)
+			)
+		)
+		(property "MPN" "SN74LVC1G86DBVR"
+			(at 123.19 124.46 0)
+			(hide yes)
+			(show_name no)
+			(do_not_autoplace no)
+			(effects
+				(font
+					(size 1.27 1.27)
+				)
+			)
+		)
+		(property "Manufacturer" "Texas Instruments"
+			(at 123.19 124.46 0)
+			(hide yes)
+			(show_name no)
+			(do_not_autoplace no)
