File: hardware/comms/kicad/transceiver.kicad_pcb (KiCad board)
At the start: 4 copper layers, 96 x 90.2 mm, 107 parts, among them J1 Conn_01x20, J2 Conn_01x20, J3 Conn_01x20, J4 Conn_Coaxial_Small, J5 Conn_Coaxial_Small, Q1 NPN, U1 MCP6022, U2 74LVC1G86, U3 PSA4-5043+, U4 ADE-1+, U6 ADL5602ARKZ-R7, Y1 Crystal_GND2, Y2 Si5351A-B-GT

Commit message: comms: checkpoint current KiCad design before ground station work
Parts:
- removed C19, C22, C24, C29, C30, C31, C32: 10p, Capacitor_SMD:C_0402_1005Metric
- removed C20, C21: 6.8p, Capacitor_SMD:C_0402_1005Metric
- removed C23: 33p, Capacitor_SMD:C_0402_1005Metric
- removed J5: Conn_Coaxial_Small, Connector_Coaxial:MMCX_Molex_73415-1471_Vertical
- removed L10, L11, L9: 82n, Inductor_SMD:L_0402_1005Metric
- removed L2, L6: 15n, Inductor_SMD:L_0402_1005Metric
- removed the TP1 at (127.2, 103.6)
- removed the TP2 at (124.2, 114.7)
- removed U1: MCP6022, Vault:SLAB-MSOP-10_N
- added C102: 100p, Capacitor_SMD:C_0402_1005Metric, F.Cu at (135.8, 132.8)
- added C103: 1u, Capacitor_SMD:C_0603_1608Metric, F.Cu at (127.0, 131.8)
- added C104: 1u, Capacitor_SMD:C_0603_1608Metric, F.Cu at (127.2, 130.0)
- added C105: 100n, Capacitor_SMD:C_0402_1005Metric, F.Cu at (139.0, 135.1)
- added C106: 100n, Capacitor_SMD:C_0402_1005Metric, F.Cu at (134.1, 134.9)
- added C55: 3.9p, Capacitor_SMD:C_0402_1005Metric, F.Cu at (146.1, 132.0)
- added C56: 9.1p, Capacitor_SMD:C_0402_1005Metric, F.Cu at (148.6, 132.4)
- added C60: 1.6p, Capacitor_SMD:C_0402_1005Metric, F.Cu at (149.2, 131.0)
- added C64: 9.1p, Capacitor_SMD:C_0402_1005Metric, F.Cu at (150.7, 132.5)
- added C67: 3.9p, Capacitor_SMD:C_0402_1005Metric, F.Cu at (152.2, 132.0)
- added C75: 100n, Capacitor_SMD:C_0402_1005Metric, F.Cu at (158.9, 131.8)
- added C8: 100nF, Capacitor_SMD:C_0805_2012Metric, F.Cu at (119.3, 148.8)
- added C81: 8.2p, Capacitor_SMD:C_0402_1005Metric, F.Cu at (143.0, 124.9)
- added C82: 100n, Capacitor_SMD:C_0402_1005Metric, F.Cu at (154.1, 116.3)
- added C85: 8.2p, Capacitor_SMD:C_0402_1005Metric, F.Cu at (155.3, 117.6)
- added C86: 3.9p, Capacitor_SMD:C_0402_1005Metric, F.Cu at (161.2, 116.3)
- added C87: 9.1p, Capacitor_SMD:C_0402_1005Metric, F.Cu at (130.9, 126.1)
- added C89: 1.6p, Capacitor_SMD:C_0402_1005Metric, F.Cu at (132.3, 126.6)
- added C9: 100nF, Capacitor_SMD:C_0805_2012Metric, F.Cu at (119.3, 133.8)
- added C90: 9.1p, Capacitor_SMD:C_0402_1005Metric, F.Cu at (162.7, 116.8)
- added C91: 1.6p, Capacitor_SMD:C_0402_1005Metric, F.Cu at (165.5, 116.3)
- added C92: 9.1p, Capacitor_SMD:C_0402_1005Metric, F.Cu at (130.9, 128.2)
- added C94: 3.9p, Capacitor_SMD:C_0402_1005Metric, F.Cu at (132.4, 128.6)
- added C95: 9.1p, Capacitor_SMD:C_0402_1005Metric, F.Cu at (166.9, 116.8)
- added C97: 3.9p, Capacitor_SMD:C_0402_1005Metric, F.Cu at (169.7, 116.3)
- added C98: 1.6p, Capacitor_SMD:C_0402_1005Metric, F.Cu at (140.9, 126.1)
- added D15: PESD5V0F1BRLD, Diode_SMD:D_SOD-882D, F.Cu at (134.4, 132.4)
- added JP1: Jumper_2_Open, Connector_PinHeader_2.54mm:PinHeader_1x02_P2.54mm_Vertical, F.Cu at (118.0, 136.6)
- added JP2: Jumper_2_Open, Connector_PinHeader_2.54mm:PinHeader_1x02_P2.54mm_Vertical, F.Cu at (118.1, 121.2)
- added L18: 15n, Inductor_SMD:L_0402_1005Metric, F.Cu at (156.0, 116.3)
- added L20: 10n, Inductor_SMD:L_0402_1005Metric, F.Cu at (164.1, 116.8)
- added L22: 10n, Inductor_SMD:L_0402_1005Metric, F.Cu at (168.3, 116.8)
- added Q4: 2SC3356, Package_TO_SOT_SMD:SOT-23, F.Cu at (158.3, 118.0)
- added R33: 47k, Resistor_SMD:R_0402_1005Metric, F.Cu at (155.3, 119.6)
- added R35: 10k, Resistor_SMD:R_0402_1005Metric, F.Cu at (142.7, 132.5)
- added R36: 10k, Resistor_SMD:R_0402_1005Metric, F.Cu at (137.5, 134.8)
- added R37: 10k, Resistor_SMD:R_0402_1005Metric, F.Cu at (127.9, 128.8)
- added R38: 100k, Resistor_SMD:R_0402_1005Metric, F.Cu at (171.0, 131.2)
- added R38: 100k, R_0402_1005Metric, F.Cu at (171.0, 130.1)
- added R39: 100k, R_0402_1005Metric, F.Cu at (179.0, 125.0)
- added R39: 100k, Resistor_SMD:R_0402_1005Metric, F.Cu at (173.0, 131.3)
- added R5: 120R, Resistor_SMD:R_0805_2012Metric, F.Cu at (119.3, 139.3)
- added R6: 120R, Resistor_SMD:R_0805_2012Metric, F.Cu at (119.3, 124.1)
- added U11: PE4259, Package_TO_SOT_SMD:SOT-363_SC-70-6, F.Cu at (135.8, 135.3)
- added U12: TLV75530PDBVR, Package_TO_SOT_SMD:SOT-23-5, F.Cu at (130.4, 130.7)
- added U13: SN74LVC1G17DBVR, Package_TO_SOT_SMD:SOT-23-5, F.Cu at (140.2, 133.0)
- added U2: SN65HVD230, Package_SO:SOIC-8_3.9x4.9mm_P1.27mm, F.Cu at (119.3, 144.1)
- added U3: SN65HVD230, Package_SO:SOIC-8_3.9x4.9mm_P1.27mm, F.Cu at (119.3, 128.8)
- added U5: MCP6022, Package_SO:SOIC-8_3.9x4.9mm_P1.27mm, F.Cu at (174.1, 124.7)
- C100: renamed from C13; value 6.8p -> 9.1p
- C101: renamed from C11; value 10p -> 3.9p
- C58: renamed from C43; footprint Vault:FP-EEH-D-MFG -> Ember_RF:CP_Elec_Panasonic_D_6.3x5.8
- C59: renamed from C49; footprint Vault:FP-EEH-D-MFG -> Ember_RF:CP_Elec_Panasonic_D_6.3x5.8
- C83: renamed from C33; value 100n -> 1n
- C84: renamed from C9; value 10p -> 3.9p
- C93: renamed from C10; value 10p -> 3.9p
- C96: renamed from C12; value 6.8p -> 9.1p
- H1, H2: footprint Vault:SAMTEC_ESQ-126-37-G-D -> Ember_RF:Samtec_ESQ-126-39-G-D_2x26_P2.54mm
- J6: renamed from J1; footprint Vault:FP-ESQ-120-14-G-S-MFG -> Connector_PinHeader_2.54mm:PinHeader_1x20_P2.54mm_Vertical
- J7: renamed from J2; footprint Vault:FP-ESQ-120-14-G-S-MFG -> Connector_PinHeader_2.54mm:PinHeader_1x20_P2.54mm_Vertical
- J8: renamed from J3; footprint Vault:FP-ESQ-120-14-G-S-MFG -> Connector_PinHeader_2.54mm:PinHeader_1x20_P2.54mm_Vertical
- L12, L13: value 68n -> 10n; footprint Vault:Chip2PinSM127P600-8N -> Inductor_SMD:L_0402_1005Metric
- L16: renamed from L14; value 1u -> 220n; footprint Inductor_SMD:L_0805_2012Metric -> Ember_RF:L_Coilcraft_0805HP
- L17: renamed from L1; value 220n -> 15n; footprint Inductor_SMD:L_0805_2012Metric -> Inductor_SMD:L_0402_1005Metric
- L19: renamed from L7; value 15n -> 10n
- L21: renamed from L8; value 15n -> 10n
- L23: renamed from L3; value 15n -> 10n
- L24: renamed from L4; value 15n -> 10n
- Q3: renamed from Q1; value NPN -> 2SC3356
- R3: renamed from R1; footprint Vault:RESC1005X40X25NL05T10 -> Resistor_SMD:R_0402_1005Metric
- R4: renamed from R2; footprint Vault:RESC1005X40X25NL05T10 -> Resistor_SMD:R_0402_1005Metric
- TP1: renamed from TP3; footprint Vault:TP06R -> TestPoint:TestPoint_Pad_D1.0mm
- TP2: renamed from TP4; footprint Vault:TP06R -> TestPoint:TestPoint_Pad_D1.0mm
- TP3: renamed from TP5; footprint Vault:TP06R -> TestPoint:TestPoint_Pad_D1.0mm
- TP4: renamed from TP6; footprint Vault:TP06R -> TestPoint:TestPoint_Pad_D1.0mm
- TP5: renamed from TP7; footprint Vault:TP06R -> TestPoint:TestPoint_Pad_D1.0mm
- TP6: renamed from TP8; footprint Vault:TP06R -> TestPoint:TestPoint_Pad_D1.0mm
- U7: renamed from U2; footprint Vault:FP-DBV0005A-MFG -> Package_TO_SOT_SMD:SOT-23-5
- U9: renamed from U3; footprint Package_TO_SOT_SMD:SOT-343_SC-70-4 -> Ember_RF:PSA4-5043_MMM1362
- Y1: value Crystal_GND2 -> 25MHz
- moved C65 80.2 mm to (139.5, 116.9), turned to -90 degrees
- moved Y2 56.7 mm to (150.8, 125.2), turned to -90 degrees
- moved C88 49.0 mm to (172.0, 119.9), turned to -90 degrees
- moved H2 31.8 mm to (106.9, 104.4), turned to 180 degrees
- moved H1 31.8 mm to (111.9, 104.4), turned to 180 degrees
- moved J6 24.1 mm to (184.6, 96.1), turned to -90 degrees
- moved J7 24.1 mm to (184.6, 113.9), turned to -90 degrees
- moved J8 24.1 mm to (190.5, 129.1), turned to 180 degrees
- moved L13 21.9 mm to (149.7, 132.5), turned to -90 degrees
- moved L12 21.4 mm to (147.6, 132.4), turned to -90 degrees
- moved U8 20.1 mm to (135.0, 124.5), turned to 180 degrees
- moved U9 19.5 mm to (154.5, 130.8), turned to -90 degrees
- moved C76 12.4 mm to (135.0, 119.4)
- moved C58 12.0 mm to (125.3, 108.8)
- moved C99 10.6 mm to (159.6, 123.2), turned to 0 degrees
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- renumbered C4 to C2, C5 to C3, C6 to C4, C7 to C5, C39 to C57, C2 to C6, C42 to C61, C48 to C62, C40 to C63, C25 to C65, C15 to C66, C50 to C68, C38 to C69, C3 to C7, C51 to C70, C17 to C71, C41 to C72, C14 to C73, C52 to C74, C18 to C76, C35 to C77, C53 to C78, C27 to C79, C16 to C80, C44 to C88, C34 to C99, D6 to D10, D7 to D11, D3 to D12, D4 to D13, D2 to D14, D1 to D8, D5 to D9, J4 to J9, L5 to L15, R3 to R1, R4 to R2, R11 to R20, R12 to R21, R14 to R22, R15 to R23, R16 to R24, R6 to R25, R17 to R26, R5 to R27, R10 to R28, R13 to R29, R9 to R30, R18 to R31, R8 to R32, R7 to R34, U4 to U10, U6 to U8
Connections:
- net /3V3_IND renamed /Digital Control/3V3_IND
- net /ADC_VREF renamed /Digital Control/ADC_VREF
- net /CLK0_OUT renamed CLK0_OUT
- net /CLK1_OUT renamed CLK1_OUT
- net /GPIO0 renamed /Digital Control/GPIO0
- net /GPIO1 renamed /Digital Control/GPIO1
- net /GPIO13 renamed /Digital Control/GPIO13
- net /GPIO22 renamed /Digital Control/GPIO22
- net /RUN_RESET renamed /Digital Control/RUN_RESET
- net /RX_ACTIVE renamed /Digital Control/RX_ACTIVE
- net /RX_BASEBAND renamed RX_BASEBAND
- net /RX_IF renamed RX_IF
- net /TX_437 renamed TX_437
- net /TX_ACTIVE renamed /Digital Control/TX_ACTIVE
- net /VBAT renamed /Connectors/VBAT
- C69 pad 1: Net-(U1B-+) -> /RX Chain/RX_AMP_IN
- C72 pad 2: Net-(U1B-+) -> /RX Chain/VREF_RX
- C73 pad 1: Net-(Q1-B) -> Net-(Q3-B)
- C73 pad 2: /BPSK_145 -> /TX Chain/RF_TX_BPSK_145
- C83 pad 1: Net-(C22-Pad1) -> Net-(Q4-B)
- C93 pad 1: /TRIPLER_OUT -> TRIPLER_OUT
- D14 pad 1: /PICO_VSYS -> PICO_VSYS
- H1 pad 16: /COMMS_IRQ -> unconnected-(H1-Pin_16-Pad16)
- H1 pad 21: /SPI_COMMS_SCK -> unconnected-(H1-Pin_21-Pad21)
- H1 pad 22: /SPI_COMMS_MISO -> unconnected-(H1-Pin_22-Pad22)
- H1 pad 23: /SPI_COMMS_MOSI -> unconnected-(H1-Pin_23-Pad23)
- H1 pad 24: /SPI_COMMS_CS_N -> unconnected-(H1-Pin_24-Pad24)
- J6 pad 10: /SPI_COMMS_MOSI -> unconnected-(J6-Pin_10-Pad10)
- J6 pad 19: /GPIO14 -> /Digital Control/CAN_B_RX
- J6 pad 20: /GPIO15 -> /Digital Control/CAN_B_TX
- J6 pad 5: /COMMS_IRQ -> unconnected-(J6-Pin_5-Pad5)
- J6 pad 6: /SPI_COMMS_MISO -> unconnected-(J6-Pin_6-Pad6)
- J6 pad 7: /SPI_COMMS_CS_N -> unconnected-(J6-Pin_7-Pad7)
- J6 pad 9: /SPI_COMMS_SCK -> unconnected-(J6-Pin_9-Pad9)
- J7 pad 14: /I2C_SCL -> I2C_SCL
- J7 pad 15: /I2C_SDA -> I2C_SDA
- J7 pad 16: unconnected-(J2-Pin_16-Pad16) -> /Digital Control/CAN_A_TX
- J7 pad 17: unconnected-(J2-Pin_17-Pad17) -> /Digital Control/CAN_A_RX
- J7 pad 2: /PICO_VSYS -> PICO_VSYS
- J7 pad 20: /BPSK_DATA -> BPSK_DATA
- J8 pad 18: /GPIO14 -> unconnected-(J8-Pin_18-Pad18)
- J8 pad 19: /GPIO15 -> unconnected-(J8-Pin_19-Pad19)
- J9 pad 1: /TX_OUT -> ANT
- L12 pad 1: Net-(C22-Pad1) -> Net-(C55-Pad2)
- L12 pad 2: Net-(C23-Pad1) -> GND
- L13 pad 1: Net-(C23-Pad1) -> Net-(C60-Pad2)
- L13 pad 2: Net-(U4-LO) -> GND
- L16 pad 2: Net-(U4-RF) -> Net-(U9-OUT_DC)
- L17 pad 2: /TRIPLER_OUT -> TRIPLER_OUT
- Q3 pad 1: /TRIPLER_OUT -> Net-(Q3-B)
- Q3 pad 2: Net-(Q1-B) -> GND
- Q3 pad 3: GND -> TRIPLER_OUT
- R1 pad 2: /I2C_SDA -> I2C_SCL
- R2 pad 2: /I2C_SCL -> I2C_SDA
- R25 pad 1: /BPSK_DATA -> BPSK_DATA
- R27 pad 1: Net-(Q1-B) -> Net-(Q3-B)
- R28 pad 2: Net-(R10-Pad2) -> /RX Chain/VREF_RX
- R29 pad 1: Net-(R10-Pad2) -> /RX Chain/VREF_RX
- R30 pad 2: GND -> /RX Chain/VREF_RX
- TP2 pad 1: /BPSK_145 -> BPSK_DATA
- TP3 pad 1: /TRIPLER_OUT -> TRIPLER_OUT
- U10 pad 3: Net-(U4-RF) -> Net-(U10-RF)
- U10 pad 6: Net-(U4-LO) -> Net-(U10-LO)
- U7 pad 4: /BPSK_145 -> /TX Chain/RF_TX_BPSK_145
- U9 pad 1: Net-(C30-Pad2) -> Net-(U9-OUT_DC)
- U9 pad 3: Net-(U4-RF) -> Net-(U9-IN)
- U9 pad 4: (no net) -> GND
- Y1 pad 4: (no net) -> GND
- Y2 pad 4: /I2C_SCL -> I2C_SCL
- Y2 pad 5: /I2C_SDA -> I2C_SDA
Routing:
- net /COMMS_IRQ: track 74.3 -> 0.00 mm
- net /SPI_COMMS_MISO: track 68.2 -> 0.00 mm
- net /SPI_COMMS_CS_N: track 65.2 -> 0.00 mm
- net +5V: track 10.4 -> 73.8 mm, vias 13 -> 11
- net /GPIO15: track 59.9 -> 0.00 mm
- net /Digital Control/CAN_A_TX: track 0.00 -> 57.5 mm, vias 0 -> 1
- net /SPI_COMMS_SCK: track 57.4 -> 0.00 mm
- net /GPIO14: track 56.6 -> 0.00 mm
- net /SPI_COMMS_MOSI: track 53.6 -> 0.00 mm
- net /Digital Control/CAN_A_RX: track 0.00 -> 51.0 mm, vias 0 -> 1
- net /Digital Control/CAN_B_TX: track 0.00 -> 44.2 mm, vias 0 -> 1
- net /Digital Control/CAN_B_RX: track 0.00 -> 43.3 mm, vias 0 -> 1
- net GND: track 23.0 -> 61.9 mm, vias 76 -> 79
- net CAN_B_L: track 0.00 -> 31.8 mm, vias 0 -> 2
- net /RX Chain/VREF_RX: track 0.00 -> 27.5 mm, vias 0 -> 5
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- removed copper zone on In2.Cu, net +3V3
- removed copper zone on F.Cu, net +5V_CON
- removed copper zone on F.Cu, net GND
- removed copper zone on F.Cu, net Net-(Q1-B)
Other:
- outline, holes or cut-outs redrawn
