File: hardware/comms/kicad/transceiver.kicad_pcb (KiCad board)
At the start: 4 copper layers, 96 x 90.2 mm, 161 parts, among them J6 Conn_01x20, J7 Conn_01x20, J8 Conn_01x20, J9 Conn_Coaxial_Small, Q3 2SC3356, Q4 2SC3356, U1 MCP25625-E/SS, U10 ADE-1+, U11 PE4259, U12 TLV73330PDBVR, U13 SN74LVC1G17DBVR, U14 SN74LVC1G08DBVR, U15 LM73100RPWR, U4 MCP25625-E/SS, U5 MCP6022, U7 74LVC1G86, U8 ADL5602ARKZ-R7, U9 PSA4-5043+, Y1 25MHz, Y2 Si5351A-B-GT, Y3 16MHz, Y4 16MHz

Commit message: Preserve purchased Y24 transceiver design and fabrication release
Archive the exact October 4 source and manufacturing artifacts, with H1/H2
connector models and final review evidence. Record payment and the unresolved
J9 hole-tolerance review separately from the immutable preview manifest.

Verified all 10 source hashes, 45 artifact hashes/sizes and the model hash.
No KiCad design changes or new electrical validation in this checkpoint.
Routing:
- net /Digital Control/ADC_VREF: track 26.2 -> 34.8 mm
- net +5V: track 261.2 -> 268.7 mm
- net /Digital Control/RUN_RESET: track 40.8 -> 45.3 mm
- net /Digital Control/GPIO22: track 42.4 -> 46.1 mm
- net /RX Chain/VREF_RX: track 30.1 -> 26.7 mm
- net /Digital Control/GPIO13: track 68.3 -> 70.7 mm
- net +3V3: track 305.6 -> 303.4 mm
- net CLK1_OUT: track 8.09 -> 6.24 mm
- net Net-(Q4-B): track 5.85 -> 4.47 mm
- net Net-(C65-Pad1): track 7.44 -> 8.78 mm
- net RX_BASEBAND: track 15.9 -> 14.9 mm
- net TX_ACTIVE: track 59.0 -> 59.6 mm
- net /RX Chain/RX_AMP_IN: track 14.2 -> 13.7 mm
- net Net-(U10-IF): track 9.86 -> 10.4 mm
