File: hardware/comms/kicad/Digital_Control.kicad_sch (KiCad schematic)
At the start: 17 parts, among them J6 Conn_01x20, J7 Conn_01x20, J8 Conn_01x20, U2 SN65HVD230, U3 SN65HVD230

Commit message: Complete dual-CAN transceiver hardware prototype
Preserve the current transceiver schematics, PCB, libraries and validation evidence as a focused hardware review against main.
Parts:
- removed U2, U3: SN65HVD230, Package_SO:SOIC-8_3.9x4.9mm_P1.27mm, symbol Interface_CAN_LIN:SN65HVD230
- added C107, C108, C109, C110, C111, C112, C113, C114: 100nF, Capacitor_SMD:C_0603_1608Metric, symbol Device:C_Small
- added R40, R41, R42, R43, R44, R45: 10k, Resistor_SMD:R_0603_1608Metric, symbol Device:R
- added U1, U4: MCP25625-E/SS, Package_SO:SSOP-28_5.3x10.2mm_P0.65mm, symbol Interface_CAN_LIN:MCP25625x-x-SS
- added Y3, Y4: 16MHz, Oscillator:Oscillator_SMD_SiT_PQFN-4Pin_7.0x5.0mm, symbol Oscillator:SiT8008xx-8x-xxE
- C8, C9: LCSC Part # (none) -> C1711; MPN (none) -> CL21B104KBCNNNC; Manufacturer (none) -> Samsung Electro-Mechanics; Manufacturer Part # (none) -> CL21B104KBCNNNC
- J6, J7, J8: Assembly (none) -> DNP; LCSC Part # (none) -> C50981; MPN (none) -> 2.54-1*20P; Manufacturer (none) -> BOOMELE; Manufacturer Part # (none) -> 2.54-1*20P
- JP1, JP2: Assembly (none) -> Hand solder; Assembly Notes (none) -> Header only; fit 2.54mm shunt only where CAN termination is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; LCSC Part # (none) -> C86471; MPN (none) -> 826629-2; Manufacturer (none) -> TE Connectivity; Manufacturer Part # (none) -> 826629-2
- R5, R6: LCSC Part # (none) -> C17437; MPN (none) -> 0805W8F1200T5E; Manufacturer (none) -> UNI-ROYAL; Manufacturer Part # (none) -> 0805W8F1200T5E
Connections:
- net GND: now also C107.2, C108.2, C109.2, C110.2, C111.2, C112.2, C113.2, C114.2, U1.10 (GND), U1.26 (V_{SS}), U4.10 (GND), U4.26 (V_{SS}), Y3.2 (GND), Y4.2 (GND)
- net CAN_SPI_MOSI: now reaches J6.10 (Pin_10)
- net CAN_SPI_MOSI: now also U1.15 (SI), U4.15 (SI)
- net CAN_A_RESETn: now reaches J6.11 (Pin_11)
- net CAN_A_RESETn: now also C110.1, R42.2, U1.18 (~{RESET})
- net CAN_B_RESETn: now reaches J6.12 (Pin_12)
- net CAN_B_RESETn: now also C114.1, R45.2, U4.18 (~{RESET})
- net CAN_A_STBY: now reaches J6.4 (Pin_4)
- net CAN_A_STBY: now also R41.2, U1.5 (STBY)
- net CAN_B_STBY: now reaches J6.5 (Pin_5)
- net CAN_B_STBY: now also R44.2, U4.5 (STBY)
- net CAN_SPI_MISO: now reaches J6.6 (Pin_6)
- net CAN_SPI_MISO: now also U1.16 (SO), U4.16 (SO)
- net CAN_SPI_SCK: now reaches J6.9 (Pin_9)
- net CAN_SPI_SCK: now also U1.14 (SCK), U4.14 (SCK)
- net CAN_A_H renamed CAN_A_P
- net CAN_A_P: now also U1.4 (CANH)
- net CAN_A_L renamed CAN_A_N
- net CAN_A_N: now also U1.3 (CANL)
- net CAN_A_RX renamed CAN_A_INTn
- net CAN_A_INTn: now also U1.13 (~{INT})
- net CAN_A_TX renamed CAN_B_INTn
- net CAN_B_INTn: now also U4.13 (~{INT})
- net CAN_B_H renamed CAN_B_P
- net CAN_B_P: now also U4.4 (CANH)
- net CAN_B_L renamed CAN_B_N
- net CAN_B_N: now also U4.3 (CANL)
- net CAN_B_RX renamed CAN_A_CSn
- net CAN_A_CSn: now also R40.2, U1.17 (~{CS})
- net CAN_B_TX renamed CAN_B_CSn
- net CAN_B_CSn: now also R43.2, U4.17 (~{CS})
- net GPIO14: no longer names the net of J8.18 (Pin_18)
- net GPIO15: no longer names the net of J8.19 (Pin_19)
- net VCC_3V3 renamed +3V3
- net +3V3: now also C107.1, C109.1, C111.1, C113.1, R40.1, R41.1, R42.1, R43.1, R44.1, R45.1, U1.1 (V_{IO}), U1.19 (V_{DD}), U1.23 (~{Tx0RTS}), U1.6 (~{Tx1RTS}), U1.7 (~{Tx2RTS}), U4.1 (V_{IO}), U4.19 (V_{DD}), U4.23 (~{Tx0RTS}), U4.6 (~{Tx1RTS}), U4.7 (~{Tx2RTS}), Y3.1 (OE), Y3.4 (Vdd), Y4.1 (OE), Y4.4 (Vdd)
- new net +5V: C108.1, C112.1, U1.27 (V_{DDA}), U4.27 (V_{DDA})
- new net CAN_A_CLK: U1.9 (OSC1), Y3.3 (OUT)
- new net CAN_A_RXD: U1.21 (RxCAN), U1.28 (R_{XD})
- new net CAN_A_TXD: U1.20 (TxCAN), U1.24 (T_{XD})
- new net CAN_B_CLK: U4.9 (OSC1), Y4.3 (OUT)
- new net CAN_B_RXD: U4.21 (RxCAN), U4.28 (R_{XD})
- new net CAN_B_TXD: U4.20 (TxCAN), U4.24 (T_{XD})
- no-connect marks 21 -> 26
Other:
- note added: "A controls"
- note added: "B controls"
- note added: "CAN A - MCP25625 controller + transceiver"
- note added: "CAN B - MCP25625 controller + transceiver"
- note added: "Default inactive: CS, STBY and RESET pulled high. Firmware drives STBY low after configuring each channel."
- note added: "Fit termination jumper only at a CAN bus endpoint."
- note added: "Place separate 100nF at VDD, VIO, VDDA and each oscillator. 5V budget: up to 70mA per active CAN channel. TXD/RXD loop nets connect controller to integrated transceiver."
- note added: "SPI0 master: GP4 MISO, GP6 SCK, GP7 MOSI A/B CS: GP14/15; IRQ: GP18/19 A/B STBY: GP2/3; RESET: GP8/9 16MHz clocks; dual-instance firmware port required."
- note removed: "CAN Transceivers"
- moved on the sheet: C8, C9, JP1, JP2, R5, R6
