File: hardware/eps/studies/recovery_5v/recovery_5v.kicad_sch (KiCad schematic)
At the start: 28 parts, among them U1 TPS 552872

Commit message: Resolve recovery component identities and startup design constraints
Parts:
- C1: Dielectric (none) -> X8L; MFG P/N (none) -> GCM188L81H104KA57D; PackageSize (none) -> 0603; Review status (none) -> EVM reference; effective capacitance acceptance open; Tolerance (none) -> 10%; Voltage (none) -> 50 V
- C10, C11, C12, C9: Dielectric (none) -> X7R; MFG P/N (none) -> CGA6P3X7R1E226M250AB; PackageSize (none) -> 1210; Review status (none) -> Development selection; application qualification open; Tolerance (none) -> 20%; Voltage (none) -> 25 V
- C13, C14, C15: Dielectric (none) -> Hybrid aluminum; Height (none) -> 7.7 mm nominal; tolerance/mechanical acceptance open; MFG P/N (none) -> EEHZK1V101XP; PackageSize (none) -> 6.3 x 7.7 mm; Review status (none) -> Development selection; application qualification open; Tolerance (none) -> 20%; Voltage (none) -> 35 V
- C16, C8: Dielectric (none) -> X7R; MFG P/N (none) -> CGA2B3X7R1H104K050BB; PackageSize (none) -> 0402; Review status (none) -> Development selection; application qualification open; Tolerance (none) -> 10%; Voltage (none) -> 50 V
- C17: footprint Capacitor_SMD:C_0603_1608Metric -> Capacitor_SMD:C_1206_3216Metric; Dielectric (none) -> C0G; MFG P/N (none) -> GRM31C5C1H753JA01L; PackageSize (none) -> 1206; Review status (none) -> Development selection; application qualification open; Tolerance (none) -> 5%; Voltage (none) -> 50 V
- C18: Dielectric (none) -> C0G; MFG P/N (none) -> GRM1885C1H301JA01D; PackageSize (none) -> 0603; Review status (none) -> Development selection; application qualification open; Tolerance (none) -> 5%; Voltage (none) -> 50 V
- C2: Dielectric (none) -> X8L; MFG P/N (none) -> GCM188L81H104KA57D; PackageSize (none) -> 0603; Review status (none) -> Development selection; application qualification open; Tolerance (none) -> 10%; Voltage (none) -> 50 V
- C3, C4, C5, C6: Dielectric (none) -> X7R; MFG P/N (none) -> CGA5L1X7R1H106K160AC; PackageSize (none) -> 1206; Review status (none) -> Development selection; application qualification open; Source status (none) -> TI EVM BOM reference; full effective-capacitance acceptance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; Tolerance (none) -> 10%; Voltage (none) -> 50 V
- C7: Dielectric (none) -> Hybrid aluminum; Height (none) -> 10.2 mm nominal; tolerance/mechanical acceptance open; MFG P/N (none) -> EEHZA1H680P; PackageSize (none) -> 8 x 10.2 mm; Review status (none) -> Development selection; application qualification open; Tolerance (none) -> 20%; Voltage (none) -> 50 V
- L1: value 10u -> 6u8; footprint (none) -> Inductor_SMD:L_Coilcraft_XAL7070-XXX; DCR (none) -> 19.6 mOhm maximum at 25 C; Height (none) -> 7.0 mm family reference; direct drawing verification open; MFG P/N (none) -> XAL7070-682MEC; PackageSize (none) -> XAL7070; Rated current (none) -> 6.8 A reference, 20 C rise at 25 C; not application rating; Review status (none) -> Development selection; hot current/fault and thermal accept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; Saturation current (none) -> 12.8 A typical, 30% L drop at 25 C; Tolerance (none) -> 20%
- R1: MFG P/N (none) -> TNPW060339K2BEEA; PackageSize (none) -> 0603; Power (none) -> 0.11 W @70 C general mode; Review status (none) -> Development selection; ordering-code construction from manu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; TCR (none) -> 25 ppm/K; Tolerance (none) -> 0.1%
- R2: MFG P/N (none) -> TNPW060316K9BEEA; PackageSize (none) -> 0603; Power (none) -> 0.11 W @70 C general mode; Review status (none) -> Development selection; ordering-code construction from manu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; TCR (none) -> 25 ppm/K; Tolerance (none) -> 0.1%
- R3: MFG P/N (none) -> TNPW060349K3BEEA; PackageSize (none) -> 0603; Power (none) -> 0.11 W @70 C general mode; Review status (none) -> Development selection; ordering-code construction from manu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; TCR (none) -> 25 ppm/K; Tolerance (none) -> 0.1%
- R4: MFG P/N (none) -> CRF1206-FZ-R020ELF; PackageSize (none) -> 1206; Power (none) -> 1 W @70 C; TCR (none) -> 50 ppm/K; Tolerance (none) -> 1%
- R5: MFG P/N (none) -> TNPW060331K6BEEA; PackageSize (none) -> 0603; Power (none) -> 0.11 W @70 C general mode; Review status (none) -> Development selection; ordering-code construction from manu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; TCR (none) -> 25 ppm/K; Tolerance (none) -> 0.1%
- R6, R8: MFG P/N (none) -> TNPW060310K0BEEA; PackageSize (none) -> 0603; Power (none) -> 0.11 W @70 C general mode; Review status (none) -> Development selection; ordering-code construction from manu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; TCR (none) -> 25 ppm/K; Tolerance (none) -> 0.1%
- R7: MFG P/N (none) -> TNPW06033K74BEEA; PackageSize (none) -> 0603; Power (none) -> 0.11 W @70 C general mode; Review status (none) -> Development selection; ordering-code construction from manu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; TCR (none) -> 25 ppm/K; Tolerance (none) -> 0.1%

Commit message: Add approved Panasonic recovery bulk capacitor footprints
Parts:
- C13, C14, C15: footprint (none) -> Ember_EPS_Recovery:Panasonic_CP_D8_6.3x7.7mm_REVIEW; Footprint review (none) -> Manufacturer land geometry query-back/render checked; assem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
- C7: footprint (none) -> Ember_EPS_Recovery:Panasonic_CP_F_8x10.2mm_REVIEW; Footprint review (none) -> Manufacturer land geometry query-back/render checked; assem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
Changed lines of the file:
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@@
 			)
 		)
-		(property "Footprint" ""
+		(property "Footprint" "Ember_EPS_Recovery:Panasonic_CP_F_8x10.2mm_REVIEW"
 			(at 121.92 119.38 0)
 			(hide yes)
@@
 		)
 		(property "Voltage" "50 V"
+			(at 121.92 119.38 0)
+			(hide yes)
+			(effects
+				(font
+					(size 1.27 1.27)
+				)
+			)
+		)
+		(property "Footprint review" "Manufacturer land geometry query-back/render checked; assembly/stencil qualification open"
 			(at 121.92 119.38 0)
 			(hide yes)
@@
 			)
 		)
-		(property "Footprint" ""
+		(property "Footprint" "Ember_EPS_Recovery:Panasonic_CP_D8_6.3x7.7mm_REVIEW"
 			(at 254 144.78 0)
 			(hide yes)
@@
 		)
 		(property "Voltage" "35 V"
+			(at 254 144.78 0)
+			(hide yes)
+			(effects
+				(font
+					(size 1.27 1.27)
+				)
+			)
+		)
+		(property "Footprint review" "Manufacturer land geometry query-back/render checked; assembly/stencil qualification open"
 			(at 254 144.78 0)
 			(hide yes)
@@
 			)
 		)
-		(property "Footprint" ""
+		(property "Footprint" "Ember_EPS_Recovery:Panasonic_CP_D8_6.3x7.7mm_REVIEW"
 			(at 274.32 144.78 0)
 			(hide yes)
@@
 		)
 		(property "Voltage" "35 V"
+			(at 274.32 144.78 0)
+			(hide yes)
+			(effects
+				(font
+					(size 1.27 1.27)
+				)
+			)
+		)
+		(property "Footprint review" "Manufacturer land geometry query-back/render checked; assembly/stencil qualification open"
 			(at 274.32 144.78 0)
 			(hide yes)
@@
 			)
 		)
-		(property "Footprint" ""
+		(property "Footprint" "Ember_EPS_Recovery:Panasonic_CP_D8_6.3x7.7mm_REVIEW"
 			(at 294.64 144.78 0)
 			(hide yes)
@@
 			(at 294.64 144.78 0)
 			(hide yes)
+			(effects
+				(font
+					(size 1.27 1.27)
+				)
+			)
+		)
+		(property "Footprint review" "Manufacturer land geometry query-back/render checked; assembly/stencil qualification open"
+			(at 294.64 144.78 0)
+			(hide yes)

Commit message: Rerate recovery output bank and expose coupled protection gaps
Parts:
- added C19, C20, C21, C22: 10u, Capacitor_SMD:C_1206_3216Metric, symbol Device:C
- added C23, C24: 68u, Ember_EPS_Recovery:Panasonic_CP_F_8x10.2mm_REVIEW, symbol Device:C_Polarized
- C10, C11, C12, C9: value 22u -> 10u; footprint Capacitor_SMD:C_1210_3225Metric -> Capacitor_SMD:C_1206_3216Metric; MFG P/N CGA6P3X7R1E226M250AB -> CGA5L1X7R1H106K160AC; PackageSize 1210 -> 1206; Review status Development selection; application qualification open -> Development bank voltage correction; effective capacitance/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; Tolerance 20% -> 10%; Voltage 25 V -> 50 V
- C13, C14, C15: value 100u -> 68u; footprint Ember_EPS_Recovery:Panasonic_CP_D8_6.3x7.7mm_REVIEW -> Ember_EPS_Recovery:Panasonic_CP_F_8x10.2mm_REVIEW; Footprint review Manufacturer land geometry query-back/render checked; assem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 -> Approved Panasonic F land; pad1 positive; assembly/stencil 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; Height 7.7 mm nominal; tolerance/mechanical acceptance open -> 10.2 mm nominal; tolerance/mechanical acceptance open; MFG P/N EEHZK1V101XP -> EEHZA1H680P; PackageSize 6.3 x 7.7 mm -> 8 x 10.2 mm; Voltage 35 V -> 50 V
Connections:
- net 5V0_RECOVERY_RAW: now also C19.1, C20.1, C21.1, C22.1, C23.1, C24.1
- net GND: now also C19.2, C20.2, C21.2, C22.2, C23.2, C24.2
Other:
- moved on the sheet: C13, C14, C15
