File: hardware/eps/studies/recovery_protection/recovery_protection.kicad_sch (KiCad schematic)
At the start: 38 parts, among them Q1 IRLR2908, Q2 IRLR2908, Q3 MMBT3906LT1G, U1 LTC4364HDE-2

Commit message: Correct recovery latch timing and source MOSFET fault stress
Parts:
- added L2: 4.7u, Inductor_SMD:L_Coilcraft_XAL1010-XXX, symbol Device:L
- C9: value 100n -> 10n; MFG P/N C1210C104J1GACTU -> C1210C103J1GACTU
- R5: footprint Resistor_SMD:R_0603_1608Metric -> Resistor_SMD:R_1210_3225Metric; Film Temperature (none) -> 125 C maximum in general mode; MFG P/N TNPW060327K8BEEA -> TNPW121027K8BEEA; PackageSize 0603 -> 1210; Power 0.11 W P70 -> 0.33 W P70 general mode; Procurement Manufacturer ordering code verified; procurement confirmati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 -> Manufacturer ordering code verified; procurement and assemb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
Connections:
- net SOLAR_PERMITTED: now also L2.1; no longer D5.1 (K), Q1.2 (D), R13.1, R2.1, R5.1
- new net SRC_FILTERED: D5.1 (K), L2.2, Q1.2 (D), R13.1, R2.1, R5.1
Other:
- note added: "L2 limits source-short slew; require >=2.5 uH through fault current. C9 = 10 nF reduces linear fault energy. Bias, OV and snubber follow L2. Development screening only; hot SOA / source / magnetic qualification open."
