File: hardware/eps/studies/recovery_protection/recovery_rail_final.kicad_sch (KiCad schematic)
At the start: 43 parts, among them Q101 IRLR2908, Q102 IRLR2908, Q103 IRLR2908, Q104 IRLR2908, Q105 IRLR2908, Q106 IRLR2908, Q107 MMBT3904LT1G, Q108 MMBT3906LT1G, U2 LTC4364HDE-1

Commit message: Correct recovery latch timing and source MOSFET fault stress
Parts:
- added R115: 330, Resistor_SMD:R_1206_3216Metric, symbol Device:R
- C112: value 68n -> 10n; MFG P/N C1210C683J1GACTU -> C1210C103J1GACTU
- C119: value 220p -> 100n; MFG P/N C1210C221J1GACTU -> C1210C104J1GACTU
- R107: value 3.20k -> 3.57k; MFG P/N TNPW06033K20BEEA -> TNPW06033K57BEEA
- R108: value 1k -> 1.11k; MFG P/N TNPW06031K00BEEA -> TNPW06031K11BEEA
Connections:
- net +5V: now also R115.1
- net GND: now also R115.2
Other:
- note added: "Latch correction: 330 ohm discharge; 100 nF timer; 10 nF gate slew. Heavy loads: >=5 ms admission ramp AND >=20 ms settling; qualify rails locally. UV reset respects cooldown: allow >=10 s before heavy loads. Hot SOA remains open."
- note added: "RECOVERY RAIL: analog 5.27 V clamp, timed latch-off"
- note removed: "RECOVERY RAIL: analog 5.25 V clamp, timed latch-off"
