File: hardware/eps/verification/rev_b/charger_bms_library/disposable/charger_bms_check.kicad_pcb (KiCad board)
At the start: 2 copper layers, 0 parts

Commit message: Complete charger and BMS placed-board physical map acceptance
Parts:
- added U1: ADI_UFD-28-1EP_4x5mm_P0.5mm_Manufacturer, Ember_Charger_BMS_Review:ADI_UFD-28-1EP_4x5mm_P0.5mm_Manufacturer, F.Cu at (20.0, 20.0)
- added U2: TI_RSM0032A-32-1EP_4x4mm_P0.4mm_Manufacturer, Ember_Charger_BMS_Review:TI_RSM0032A-32-1EP_4x4mm_P0.4mm_Manufacturer, F.Cu at (35.0, 20.0)
