File: hardware/eps/rev_b/rail_protection.kicad_sch (KiCad schematic)
At the start: 44 parts, among them Q603 IRLR2908, Q604 IRLR2908, Q605 IRLR2908, Q606 IRLR2908, Q607 IRLR2908, Q608 IRLR2908, Q609 MMBT3904LT1G, Q610 MMBT3906LT1G, U601 LTC4364HDE-1

Commit message: Integrate EPS Rev B battery management development circuit
Parts:
- R614, R621: TCR 25 ppm/K -> 100 ppm/K
Changed lines of the file:
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@@
 			)
 		)
-		(property "TCR" "25 ppm/K"
+		(property "TCR" "100 ppm/K"
 			(at 299.72 176.53 0)
 			(hide yes)
@@
 			)
 		)
-		(property "TCR" "25 ppm/K"
+		(property "TCR" "100 ppm/K"
 			(at 45.72 140.97 0)
 			(hide yes)
