File: hardware/eps/rev_b/bms_protection.kicad_sch (KiCad schematic)
At the start: 44 parts, among them J200 BM07B-GHS-TBT(LF)(SN), Q200 CSD18543Q3A, Q201 CSD18543Q3A, Q202 BSS84-7-F, Q203 DMN62D2U-7, U200 BQ40Z50RSMR-R2, U201 ISO1540DR

Commit message: Integrate isolated BMS supply and MCU branch recovery controls
Connections:
- net +3V3: no longer C210.1, R218.1, R219.1, U201.8 (VCC2)
- new net 3V3_BMS_ISO: C210.1, R218.1, R219.1, U201.8 (VCC2)
Other:
- note added: "100kbit/s: side1 <=40pF, side2 <=200pF. Both sides >=3V +1ms before polling. Reserve 13.8mA IC +3.431mA pullups. Static margins only; no rail-step proof. Isolated supply is a development candidate."
- note added: "ISOLATED BUS POWER CANDIDATE 3V3_BMS_ISO now supplies ISO1540 side2 and pullups. RAW/system returns remain separate across the shunt. Prior shared-positive supply has been removed. Gauging, startup, calibration and fault/PVT acceptance OPEN."
- note removed: "100kbit/s: side1<=40pF, side2<=200pF. Both sides >=3V +1ms before polling. Reserve13.8mA IC +3.431mA pullups. Static margins only; no rail-step proof. Offset can reverse idle-current sign."
- note removed: "BUS SUPPLY PROVISIONAL Shared+3V3 positive; distinct ground returns. Raw bus current bypasses shunt measurement: up to 8.42mA state-dependent. Gauging NOT accepted. Isolated power unresolved. No whole-board galvanic power-isolation claim."
Changed lines of the file:
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@@
 		)
 	)
-	(text "BUS SUPPLY PROVISIONAL\nShared+3V3 positive;\ndistinct ground returns.\nRaw bus current bypasses\nshunt measurement: up to\n8.42mA state-dependent.\nGauging NOT accepted.\nIsolated power unresolved.\nNo whole-board galvanic\npower-isolation claim."
-		(at 365.76 111.76 0)
-		(effects
-			(font
-				(size 1.27 1.27)
-				(bold yes)
-			)
-			(justify left bottom)
-		)
-	)
-	(text "100kbit/s: side1<=40pF, side2<=200pF.\nBoth sides >=3V +1ms before polling.\nReserve13.8mA IC +3.431mA pullups.\nStatic margins only; no rail-step proof.\nOffset can reverse idle-current sign."
-		(at 340.36 144.78 0)
-		(effects
-			(font
-				(size 1.27 1.27)
-			)
-			(justify left bottom)
-		)
-	)
 	(text "Q203: low-Vth ground-gate development choice.\nReverse hotplug / cold gate / hot SOA remain open."
 		(at 273.05 111.76 0)
@@
 		)
 	)
+  (text "ISOLATED BUS POWER CANDIDATE\n3V3_BMS_ISO now supplies\nISO1540 side2 and pullups.\nRAW/system returns remain\nseparate across the shunt.\nPrior shared-positive supply\nhas been removed. Gauging,\nstartup, calibration and\nfault/PVT acceptance OPEN."
+    (at 365.76 111.76 0)
+    (effects (font (size 1.1 1.1)) (justify left top))
+  )
+  (text "100kbit/s: side1 <=40pF, side2 <=200pF.\nBoth sides >=3V +1ms before polling.\nReserve 13.8mA IC +3.431mA pullups.\nStatic margins only; no rail-step proof.\nIsolated supply is a development candidate."
+    (at 340.36 144.78 0)
+    (effects (font (size 1 1)) (justify left top))
+  )
 	(symbol
 		(lib_id "Ember_Charger_BMS_Review:BQ40Z50RSMR-R2")
@@
 			)
 		)
-		(property "Value" "+3V3"
+		(property "Value" "3V3_BMS_ISO"
 			(at 345.44 166.624 0)
 			(effects
@@
 			)
 		)
-		(property "Value" "+3V3"
+		(property "Value" "3V3_BMS_ISO"
 			(at 396.24 176.784 0)
 			(effects
@@
 			)
 		)
-		(property "Value" "+3V3"
+		(property "Value" "3V3_BMS_ISO"
 			(at 375.92 176.784 0)
 			(effects
