File: hardware/eps/rev_b/can_interfaces.kicad_sch (KiCad schematic)
At the start: 16 parts, among them J101 CAN_A_STACK_LOGICAL, J102 CAN_B_STACK_LOGICAL, U101 TCAN3413DR, U102 TCAN3413DR

Commit message: Integrate independent CAN supplies and standby-controlled latch reset
Parts:
- added R1100, R1101, R1102, R1110, R1111, R1112: 1k, Resistor_SMD:R_0603_1608Metric, symbol Device:R
- added R1103, R1113: 47k, Resistor_SMD:R_0603_1608Metric, symbol Device:R
Connections:
- net +3V3: now also R1103.1, R1113.1; no longer C104.1, C105.1, C106.1, C107.1, C108.1, C109.1, U101.3 (VCC), U101.5 (VIO), U102.3 (VCC), U102.5 (VIO)
- net EPS_CAN_A_RX: now also R1101.1, R1103.2; no longer U101.4 (RXD)
- net EPS_CAN_A_STB: now also R1102.1; no longer U101.8 (STB)
- net EPS_CAN_A_TX: now also R1100.1; no longer U101.1 (TXD)
- net EPS_CAN_B_RX: now also R1111.1, R1113.2; no longer U102.4 (RXD)
- net EPS_CAN_B_STB: now also R1112.1; no longer U102.8 (STB)
- net EPS_CAN_B_TX: now also R1110.1; no longer U102.1 (TXD)
- new net 3V3_CANA: C104.1, C105.1, C106.1, U101.3 (VCC), U101.5 (VIO)
- new net 3V3_CANB: C107.1, C108.1, C109.1, U102.3 (VCC), U102.5 (VIO)
- new net CANA_RXD: R1101.2, U101.4 (RXD)
- new net CANA_STB: R1102.2, U101.8 (STB)
- new net CANA_TXD: R1100.2, U101.1 (TXD)
- new net CANB_RXD: R1111.2, U102.4 (RXD)
- new net CANB_STB: R1112.2, U102.8 (STB)
- new net CANB_TXD: R1110.2, U102.1 (TXD)
Other:
- note added: "Development branch power: separate TPS2553 + 1 ohm rails feed VCC / VIO and local caps. TXD / STB old pullups stay on shared +3V3 before 1k series parts; RXD has MCU-side 47k pullup. STB HIGH = branch OFF (no CAN wake); LOW = normal. See CAN Branch Power sheet. Shared +3V3, GND, MCU and clock remain common failure paths; fault / PVT acceptance OPEN."
- note removed: "FAULT LIMIT: shared +3V3, GND, MCU and clock remain common paths. Independent VCC/VIO + pullup branch limiting remains a written candidate. CAN B is bus-path recovery, not independent controller/power redundancy."
